File: production/ecad/MuscleRecoveryV1/MuscleBooting.kicad_sch (KiCad schematic)
At the start: 0 parts

Commit message: Combined schematics together
Parts:
- added C6, C7: C_Small, symbol Device:C_Small
- added C8: 4.7uF, symbol Device:C_Small
- added C9: 100nF, symbol Device:C_Small
- added J4: USB_C_Receptacle_USB2.0, Connector_USB:USB_C_Plug_Molex_105444, symbol Connector:USB_C_Receptacle_USB2.0
- added Q2, Q3: AO3400A, Package_TO_SOT_SMD:SOT-23, symbol Transistor_FET:AO3400A
- added R10, R9: 5.1K, symbol Device:R_Small
- added R11, R12: R_Small, symbol Device:R_Small
- added R13: 22.1K, symbol Device:R_Small
- added R14: 47.5K, symbol Device:R_Small
- added R15, R16, R7, R8: 10K, symbol Device:R_Small
- added R17, R18: 0, symbol Device:R_Small
- added SW1, SW2: SW_Push, symbol Switch:SW_Push
- added U3: CP2102N-Axx-xQFN28, Package_DFN_QFN:QFN-28-1EP_5x5mm_P0.5mm_EP3.35x3.35mm, symbol Interface_USB:CP2102N-Axx-xQFN28
Connections:
- new net: R16.2, U3.9 (~{RST})
- new net: J4.A5 (CC1), R10.1
- new net: J4.B5 (CC2), R9.1
- new net +3.3V: C8.1, C9.1, R11.1, R12.1, R16.1, U3.6 (VDD), U3.7 (VREGIN)
- new net DTR: Q3.2 (S), R7.1, U3.28 (~{DTR})
- new net DTR_Q: Q2.1 (G), R7.2
- new net EN: C7.1, Q2.3 (D), R12.2, SW2.1
- new net GND: C6.2, C7.2, C8.2, C9.2, J4.A1 (GND), J4.A12 (GND), J4.B1 (GND), J4.B12 (GND), R10.2, R14.2, R15.2, R9.2, SW1.2, SW2.2, U3.3 (GND)
- new net IO0: C6.1, Q3.3 (D), R11.2, SW1.1
- new net RTS: Q2.2 (S), R8.1, U3.24 (~{RTS})
- new net RTS_Q: Q3.1 (G), R8.2
- new net RXD: R17.1, U3.26 (TXD)
- new net RXD0: R17.2
- new net SUS_IN: R15.1, U3.11 (~{SUSPEND})
- new net TXD: R18.1, U3.25 (RXD)
- new net TXD0: R18.2
- new net USB+: J4.A7 (D-), J4.B7 (D-), U3.4 (D+)
- new net USB-: J4.A6 (D+), J4.B6 (D+), U3.5 (D-)
- new net VBUS: J4.A4 (VBUS), J4.A9 (VBUS), J4.B4 (VBUS), J4.B9 (VBUS), R13.1
- new net VBUS_IN: R13.2, R14.1, U3.8 (VBUS)
- no-connect marks 0 -> 18
Other:
- note added: "AutoBoot Circuitry"
- note added: "DNI"
- note added: "USB-C"

Commit message: Revert "Display commit 1"
This reverts commit 52e50f7827ccbfa861bea7a8a003d131d02fed89.
Parts:
- removed R7: 10K, symbol Device:R_Small
- added IO0, TP4, VBUS1: TestPoint, symbol Connector:TestPoint
- added R40: 10K, symbol Device:R_Small
Connections:
- net DTR: now also R40.1
- net DTR_Q: now also R40.2
- net EN: now also TP4.1
- net GND: now also U3.29 (GND)
- net IO0: now also IO0.1
- net VBUS: now also VBUS1.1

Commit message: Display commit 1
Parts:
- removed IO0, TP4, VBUS1: TestPoint, symbol Connector:TestPoint
- removed R40: 10K, symbol Device:R_Small
- added R7: 10K, symbol Device:R_Small
Connections:
- net DTR: now also R7.1
- net DTR_Q: now also R7.2
- net GND: no longer U3.29 (GND)
