File: production/ecad/MuscleRecoveryV1/MuscleBooting.kicad_sch (KiCad schematic)
At the start: 25 parts, among them J4 USB_C_Receptacle_USB2.0, Q2 AO3400A, Q3 AO3400A, U3 CP2102N-Axx-xQFN28

Commit message: updated footprint assignments for ESP32 and S1-S4 to reference the folder Andy made
Parts:
- S2, S3: footprint B3F-1000:SW_B3F-1000 -> Muscle_Recovery_Footprint_Library:SW_B3F-1000
Changed lines of the file:
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@@
       (effects (font (size 1.27 1.27)))
     )
-    (property "Footprint" "B3F-1000:SW_B3F-1000" (at 115.57 154.94 0)
+    (property "Footprint" "Muscle_Recovery_Footprint_Library:SW_B3F-1000" (at 115.57 154.94 0)
       (effects (font (size 1.27 1.27)) (justify bottom) hide)
     )
@@
       (effects (font (size 1.27 1.27)))
     )
-    (property "Footprint" "B3F-1000:SW_B3F-1000" (at 155.829 153.543 0)
-      (effects (font (size 1.27 1.27)) (justify bottom) hide)
-    )
+    (property "Footprint" "Muscle_Recovery_Footprint_Library:SW_B3F-1000" (at 155.829 153.543 0)
+      (effects (font (size 1.27 1.27)) (justify bottom) hide)
+    )

Commit message: pushing current layout and other changes to be able to pull
Parts:
- removed J4: USB_C_Receptacle_USB2.0, Connector_USB:USB_C_Plug_Molex_105444, symbol Connector:USB_C_Receptacle_USB2.0
- added J5: USB4110-GF-A, USB4110-GF-A_GCT, symbol MuscleRecoverySymbolLibray:USB4110-GF-A
Connections:
- net GND: now also J5.A1-B12 (GND), J5.A12-B1 (GND)
- net USB+: now also J5.A6 (DP1), J5.B6 (DP2)
- net USB-: now also J5.A7 (DN1), J5.B7 (DN2)
- net VBUS: now also J5.A4-B9 (VBUS), J5.A9-B4 (VBUS)
- net at R10.1: now also J5.A5 (CC1)
- net at R9.1: now also J5.B5 (CC2)
- net +3.3V renamed +3V3
- no-connect marks 22 -> 21
Other:
- moved on the sheet: C8, R10, R16

Commit message: added accelerometer
Parts:
- J5: footprint USB4110-GF-A_GCT -> (none)
Changed lines of the file:
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@@
       (effects (font (size 1.524 1.524)))
     )
-    (property "Footprint" "USB4110-GF-A_GCT" (at 8.89 43.18 0)
+    (property "Footprint" "" (at 8.89 43.18 0)
       (effects (font (size 1.27 1.27) italic) hide)
     )
