File: production/ecad/MuscleRecoveryV1/MuscleBooting.kicad_sch (KiCad schematic)
At the start: 25 parts, among them J5 USB4110-GF-A, Q2 AO3400A, Q3 AO3400A, U3 CP2102N-Axx-xQFN28

Commit message: updated bom
Parts:
- J5: footprint (none) -> Muscle_Recovery_Footprint_Library:USB4110-GF-A_GCT
Changed lines of the file:
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@@
       (effects (font (size 1.524 1.524)))
     )
-    (property "Footprint" "" (at 8.89 43.18 0)
+    (property "Footprint" "Muscle_Recovery_Footprint_Library:USB4110-GF-A_GCT" (at 8.89 43.18 0)
       (effects (font (size 1.27 1.27) italic) hide)
     )
