File: production/ecad/MuscleRecoveryV1/MusclePower.kicad_sch (KiCad schematic)
At the start: 24 parts, among them IC1 LC709203FQH-01TWG, Q1 FDN340P, U1 AP1117-33, U2 MCP73831-2-OT

Commit message: Footprints added
Parts:
- removed R35: R, symbol Device:R
- BATT1: footprint (none) -> TestPoint:TestPoint_Pad_D1.5mm
- C15, C16, C17, C18, C5: footprint (none) -> Capacitor_SMD:C_0805_2012Metric
- D1, D3, D4: footprint (none) -> LED_THT:LED_D1.8mm_W3.3mm_H2.4mm
- R32, R33, R37, R38, R39, R41, R42, R43: footprint (none) -> Resistor_SMD:R_0805_2012Metric
Changed lines of the file:
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@@
       (effects (font (size 1.27 1.27)) (justify left))
     )
-    (property "Footprint" "" (at 132.715 51.435 0)
+    (property "Footprint" "Capacitor_SMD:C_0805_2012Metric" (at 132.715 51.435 0)
       (effects (font (size 1.27 1.27)) hide)
     )
@@
       (effects (font (size 1.27 1.27)))
     )
-    (property "Footprint" "" (at 149.86 49.53 0)
+    (property "Footprint" "Resistor_SMD:R_0805_2012Metric" (at 149.86 49.53 0)
       (effects (font (size 1.27 1.27)) hide)
     )
@@
       (effects (font (size 1.27 1.27)))
     )
-    (property "Footprint" "" (at 64.77 114.808 90)
+    (property "Footprint" "Resistor_SMD:R_0805_2012Metric" (at 64.77 114.808 90)
       (effects (font (size 1.27 1.27)) hide)
     )
@@
         (path "/ec7ffed6-1d2d-48f7-b073-d0a7d4b8c858"
           (reference "#PWR026") (unit 1)
-        )
-      )
-    )
-  )
-  (symbol (lib_id "Device:R") (at 59.69 92.71 0) (unit 1)
-    (in_bom yes) (on_board yes) (dnp no) (fields_autoplaced)
-    (property "Reference" "R35" (at 62.23 91.44 0)
-      (effects (font (size 1.27 1.27)) (justify left))
-    )
-    (property "Value" "R" (at 62.23 93.98 0)
-      (effects (font (size 1.27 1.27)) (justify left))
-    )
-    (property "Footprint" "" (at 57.912 92.71 90)
-      (effects (font (size 1.27 1.27)) hide)
-    )
-    (property "Datasheet" "~" (at 59.69 92.71 0)
-      (effects (font (size 1.27 1.27)) hide)
-    )
-    (pin "1")
-    (pin "2")
-    (instances
-      (project "MuscleRecoveryV1"
-        (path "/4e550305-79d2-4e4a-a502-817ebcc79f9a/648f095b-a230-48ff-8dbf-d0fbef398770"
-          (reference "R35") (unit 1)
         )
       )
@@
       (effects (font (size 1.27 1.27)))
     )
-    (property "Footprint" "" (at 64.77 117.348 90)
+    (property "Footprint" "Resistor_SMD:R_0805_2012Metric" (at 64.77 117.348 90)
       (effects (font (size 1.27 1.27)) hide)
     )
@@
       (effects (font (size 1.27 1.27)))
     )
-    (property "Footprint" "" (at 38.608 102.87 90)
+    (property "Footprint" "Resistor_SMD:R_0805_2012Metric" (at 38.608 102.87 90)
       (effects (font (size 1.27 1.27)) hide)
     )
@@
       (effects (font (size 1.27 1.27)))
     )
-    (property "Footprint" "" (at 149.86 58.42 0)
+    (property "Footprint" "Resistor_SMD:R_0805_2012Metric" (at 149.86 58.42 0)
       (effects (font (size 1.27 1.27)) hide)
     )
@@
       (effects (font (size 1.27 1.27)))
     )
-    (property "Footprint" "" (at 159.385 58.42 90)
+    (property "Footprint" "LED_THT:LED_D1.8mm_W3.3mm_H2.4mm" (at 159.385 58.42 90)
       (effects (font (size 1.27 1.27)) hide)
     )
@@
       (effects (font (size 1.27 1.27)) (justify left))
     )
-    (property "Footprint" "" (at 23.8252 111.76 0)
+    (property "Footprint" "Capacitor_SMD:C_0805_2012Metric" (at 23.8252 111.76 0)
       (effects (font (size 1.27 1.27)) hide)
     )
@@
       (effects (font (size 1.27 1.27)) (justify left))
     )
-    (property "Footprint" "" (at 41.91 118.618 90)
+    (property "Footprint" "Resistor_SMD:R_0805_2012Metric" (at 41.91 118.618 90)
       (effects (font (size 1.27 1.27)) hide)
     )
@@
       (effects (font (size 1.27 1.27)) (justify left))
     )
-    (property "Footprint" "" (at 50.8 58.42 0)
+    (property "Footprint" "Capacitor_SMD:C_0805_2012Metric" (at 50.8 58.42 0)
       (effects (font (size 1.27 1.27)) hide)
     )
@@
       (effects (font (size 1.27 1.27)) (justify right))
     )
-    (property "Footprint" "" (at 36.83 110.49 0)
+    (property "Footprint" "LED_THT:LED_D1.8mm_W3.3mm_H2.4mm" (at 36.83 110.49 0)
       (effects (font (size 1.27 1.27)) hide)
     )
@@
       (effects (font (size 1.27 1.27)) (justify left))
     )
-    (property "Footprint" "" (at 95.25 58.42 0)
+    (property "Footprint" "Capacitor_SMD:C_0805_2012Metric" (at 95.25 58.42 0)
       (effects (font (size 1.27 1.27)) hide)
     )
@@
       (effects (font (size 1.27 1.27)) (justify left))
     )
-    (property "Footprint" "" (at 202.565 48.895 0)
+    (property "Footprint" "Capacitor_SMD:C_0805_2012Metric" (at 202.565 48.895 0)
       (effects (font (size 1.27 1.27)) hide)
     )
@@
       (effects (font (size 1.27 1.27)))
     )
-    (property "Footprint" "" (at 159.385 49.53 90)
+    (property "Footprint" "LED_THT:LED_D1.8mm_W3.3mm_H2.4mm" (at 159.385 49.53 90)
       (effects (font (size 1.27 1.27)) hide)
     )
@@
       (effects (font (size 1.27 1.27)))
     )
-    (property "Footprint" "" (at 193.675 52.705 0)
+    (property "Footprint" "Resistor_SMD:R_0805_2012Metric" (at 193.675 52.705 0)
       (effects (font (size 1.27 1.27)) hide)
     )
@@
       (effects (font (size 1.27 1.27)) (justify left))
     )
-    (property "Footprint" "" (at 27.94 59.69 0)
+    (property "Footprint" "Resistor_SMD:R_0805_2012Metric" (at 27.94 59.69 0)
       (effects (font (size 1.27 1.27)) hide)
     )
@@
       (effects (font (size 1.27 1.27)) (justify left))
     )
-    (property "Footprint" "" (at 147.32 100.33 0)
-      (effects (font (size 1.27 1.27)) hide)
-    )
+    (property "Footprint" "TestPoint:TestPoint_Pad_D1.5mm" (at 147.32 100.33 0)
+      (effects (font (size 1.27 1.27)) hide)
+    )

Commit message: pushing current layout and other changes to be able to pull
Parts:
- added J9: Screw_Terminal_01x02, Connector_PinHeader_2.54mm:PinHeader_1x02_P2.54mm_Vertical, symbol Connector:Screw_Terminal_01x02
Connections:
- net +BATT: now also J9.1 (Pin_1); no longer R36.1
- net GND: now also J9.2 (Pin_2)
- net +3.3V renamed +3V3
- net +3V3: now also R36.1
Changed lines of the file:
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@@
   (junction (at 132.715 44.45) (diameter 0) (color 0 0 0 0)
-  )
-  (junction (at 81.28 96.52) (diameter 0) (color 0 0 0 0)
   )
   (junction (at 202.565 44.45) (diameter 0) (color 0 0 0 0)
@@
     (stroke (width 0) (type default))
   )
-  (wire (pts (xy 81.28 96.52) (xy 81.28 102.87))
-    (stroke (width 0) (type default))
-  )
   (wire (pts (xy 132.715 40.64) (xy 132.715 44.45))
     (stroke (width 0) (type default))
@@
     (stroke (width 0) (type default))
   )
+  (wire (pts (xy 171.45 101.6) (xy 171.45 100.33))
+    (stroke (width 0) (type default))
+  )
   (wire (pts (xy 22.86 111.76) (xy 22.86 114.3))
     (stroke (width 0) (type default))
@@
     (stroke (width 0) (type default))
   )
+  (wire (pts (xy 171.45 97.79) (xy 177.8 97.79))
+    (stroke (width 0) (type default))
+  )
   (wire (pts (xy 46.99 116.84) (xy 46.99 121.92))
     (stroke (width 0) (type default))
@@
     (stroke (width 0) (type default))
   )
-  (wire (pts (xy 81.28 96.52) (xy 97.79 96.52))
-    (stroke (width 0) (type default))
-  )
   (wire (pts (xy 27.9908 48.26) (xy 43.18 48.26))
     (stroke (width 0) (type default))
@@
     (stroke (width 0) (type default))
   )
+  (wire (pts (xy 171.45 93.98) (xy 171.45 97.79))
+    (stroke (width 0) (type default))
+  )
   (wire (pts (xy 95.25 51.7144) (xy 95.25 55.88))
     (stroke (width 0) (type default))
@@
     (stroke (width 0) (type default))
   )
+  (wire (pts (xy 171.45 100.33) (xy 177.8 100.33))
+    (stroke (width 0) (type default))
+  )
   (wire (pts (xy 202.565 51.435) (xy 202.565 66.675))
     (stroke (width 0) (type default))
@@
     (stroke (width 0) (type default))
   )
-  (wire (pts (xy 81.28 93.98) (xy 81.28 96.52))
+  (wire (pts (xy 81.28 93.98) (xy 81.28 102.87))
     (stroke (width 0) (type default))
   )
@@
     )
   )
+  (symbol (lib_id "power:+BATT") (at 171.45 93.98 0) (unit 1)
+    (in_bom yes) (on_board yes) (dnp no) (fields_autoplaced)
+    (property "Reference" "#PWR068" (at 171.45 97.79 0)
+      (effects (font (size 1.27 1.27)) hide)
+    )
+    (property "Value" "+BATT" (at 171.45 89.6112 0)
+      (effects (font (size 1.27 1.27)))
+    )
+    (property "Footprint" "" (at 171.45 93.98 0)
+      (effects (font (size 1.27 1.27)) hide)
+    )
+    (property "Datasheet" "" (at 171.45 93.98 0)
+      (effects (font (size 1.27 1.27)) hide)
+    )
+    (pin "1")
+    (instances
+      (project "MuscleRecoveryV1"
+        (path "/4e550305-79d2-4e4a-a502-817ebcc79f9a/648f095b-a230-48ff-8dbf-d0fbef398770"
+          (reference "#PWR068") (unit 1)
+        )
+      )
+      (project "Power For Muscle Recovery"
+        (path "/68ba6acb-d7b0-4091-ad4f-10769cda4f80"
+          (reference "#PWR02") (unit 1)
+        )
+      )
+      (project "New Test"
+        (path "/ec7ffed6-1d2d-48f7-b073-d0a7d4b8c858"
+          (reference "#PWR03") (unit 1)
+        )
+      )
+    )
+  )
   (symbol (lib_id "Diode:MBR1020VL") (at 36.83 53.848 180) (unit 1)
     (in_bom yes) (on_board yes) (dnp no) (fields_autoplaced)
@@
     )
   )
-  (symbol (lib_id "power:+3.3V") (at 95.25 49.53 0) (unit 1)
-    (in_bom yes) (on_board yes) (dnp no) (fields_autoplaced)
-    (property "Reference" "#PWR021" (at 95.25 53.34 0)
-      (effects (font (size 1.27 1.27)) hide)
-    )
-    (property "Value" "+3.3V" (at 95.25 44.45 0)
-      (effects (font (size 1.27 1.27)))
-    )
-    (property "Footprint" "" (at 95.25 49.53 0)
-      (effects (font (size 1.27 1.27)) hide)
-    )
-    (property "Datasheet" "" (at 95.25 49.53 0)
-      (effects (font (size 1.27 1.27)) hide)
-    )
-    (pin "1")
-    (instances
-      (project "MuscleRecoveryV1"
-        (path "/4e550305-79d2-4e4a-a502-817ebcc79f9a/648f095b-a230-48ff-8dbf-d0fbef398770"
-          (reference "#PWR021") (unit 1)
-        )
-      )
-      (project "Power For Muscle Recovery"
-        (path "/68ba6acb-d7b0-4091-ad4f-10769cda4f80"
-          (reference "#PWR06") (unit 1)
-        )
-      )
-      (project "New Test"
-        (path "/ec7ffed6-1d2d-48f7-b073-d0a7d4b8c858"
-          (reference "#PWR06") (unit 1)
-        )
-      )
-    )
-  )
   (symbol (lib_id "Device:R") (at 36.83 102.87 180) (unit 1)
     (in_bom yes) (on_board yes) (dnp no)
@@
     )
   )
+  (symbol (lib_id "Connector:Screw_Terminal_01x02") (at 182.88 97.79 0) (unit 1)
+    (in_bom yes) (on_board yes) (dnp no) (fields_autoplaced)
+    (property "Reference" "J9" (at 185.42 97.79 0)
+      (effects (font (size 1.27 1.27)) (justify left))
+    )
+    (property "Value" "Screw_Terminal_01x02" (at 185.42 100.33 0)
+      (effects (font (size 1.27 1.27)) (justify left))
+    )
+    (property "Footprint" "Connector_PinHeader_2.54mm:PinHeader_1x02_P2.54mm_Vertical" (at 182.88 97.79 0)
+      (effects (font (size 1.27 1.27)) hide)
+    )
+    (property "Datasheet" "~" (at 182.88 97.79 0)
+      (effects (font (size 1.27 1.27)) hide)
+    )
+    (pin "1")
+    (pin "2")
+    (instances
+      (project "MuscleRecoveryV1"
+        (path "/4e550305-79d2-4e4a-a502-817ebcc79f9a/648f095b-a230-48ff-8dbf-d0fbef398770"
+          (reference "J9") (unit 1)
+        )
+      )
+    )
+  )
   (symbol (lib_id "power:GND") (at 193.675 66.675 0) (unit 1)
     (in_bom yes) (on_board yes) (dnp no) (fields_autoplaced)
@@
         (path "/ec7ffed6-1d2d-48f7-b073-d0a7d4b8c858"
           (reference "#PWR029") (unit 1)
+        )
+      )
+    )
+  )
+  (symbol (lib_id "power:GND") (at 171.45 101.6 0) (unit 1)
+    (in_bom yes) (on_board yes) (dnp no) (fields_autoplaced)
+    (property "Reference" "#PWR069" (at 171.45 107.95 0)
+      (effects (font (size 1.27 1.27)) hide)
+    )
+    (property "Value" "GND" (at 171.45 106.68 0)
+      (effects (font (size 1.27 1.27)))
+    )
+    (property "Footprint" "" (at 171.45 101.6 0)
+      (effects (font (size 1.27 1.27)) hide)
+    )
+    (property "Datasheet" "" (at 171.45 101.6 0)
+      (effects (font (size 1.27 1.27)) hide)
+    )
+    (pin "1")
+    (instances
+      (project "MuscleRecoveryV1"
+        (path "/4e550305-79d2-4e4a-a502-817ebcc79f9a/648f095b-a230-48ff-8dbf-d0fbef398770"
+          (reference "#PWR069") (unit 1)
+        )
+      )
+      (project "New Test"
+        (path "/ec7ffed6-1d2d-48f7-b073-d0a7d4b8c858"
+          (reference "#PWR028") (unit 1)
         )
       )
@@
     )
   )
+  (symbol (lib_id "power:+3V3") (at 95.25 49.53 0) (unit 1)
+    (in_bom yes) (on_board yes) (dnp no) (fields_autoplaced)
+    (property "Reference" "#PWR065" (at 95.25 53.34 0)
+      (effects (font (size 1.27 1.27)) hide)
+    )
+    (property "Value" "+3V3" (at 95.25 45.085 0)
+      (effects (font (size 1.27 1.27)))
+    )
+    (property "Footprint" "" (at 95.25 49.53 0)
+      (effects (font (size 1.27 1.27)) hide)
+    )
+    (property "Datasheet" "" (at 95.25 49.53 0)
+      (effects (font (size 1.27 1.27)) hide)
+    )
+    (pin "1")
+    (instances
+      (project "MuscleRecoveryV1"
+        (path "/4e550305-79d2-4e4a-a502-817ebcc79f9a"
+          (reference "#PWR065") (unit 1)
+        )
+        (path "/4e550305-79d2-4e4a-a502-817ebcc79f9a/648f095b-a230-48ff-8dbf-d0fbef398770"
+          (reference "#PWR070") (unit 1)
+        )
+      )
+    )
+  )
   (symbol (lib_id "Device:R_Small") (at 193.675 52.705 180) (unit 1)
     (in_bom yes) (on_board yes) (dnp no)
@@
         )
       )
+    )
+  )
+  (symbol (lib_id "power:+3V3") (at 97.79 96.52 0) (unit 1)
+    (in_bom yes) (on_board yes) (dnp no) (fields_autoplaced)
+    (property "Reference" "#PWR065" (at 97.79 100.33 0)
+      (effects (font (size 1.27 1.27)) hide)
+    )
+    (property "Value" "+3V3" (at 97.79 92.075 0)
+      (effects (font (size 1.27 1.27)))
+    )
+    (property "Footprint" "" (at 97.79 96.52 0)
+      (effects (font (size 1.27 1.27)) hide)
+    )
+    (property "Datasheet" "" (at 97.79 96.52 0)
+      (effects (font (size 1.27 1.27)) hide)
+    )
+    (pin "1")
+    (instances
+      (project "MuscleRecoveryV1"
+        (path "/4e550305-79d2-4e4a-a502-817ebcc79f9a"
+          (reference "#PWR065") (unit 1)
+        )
+        (path "/4e550305-79d2-4e4a-a502-817ebcc79f9a/648f095b-a230-48ff-8dbf-d0fbef398770"
+          (reference "#PWR062") (unit 1)
+        )
+      )

Commit message: added accelerometer to layout
Connections:
- net +BATT: now also C17.2; no longer C17.1
- net GND: now also C17.1; no longer C17.2
Other:
- moved on the sheet: C17
Changed lines of the file:
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@@
   (junction (at 95.25 51.7144) (diameter 0) (color 0 0 0 0)
+  )
+  (junction (at 81.28 97.79) (diameter 0) (color 0 0 0 0)
   )
   (junction (at 50.8 54.0004) (diameter 0) (color 0 0 0 0)
@@
     (stroke (width 0) (type default))
   )
-  (wire (pts (xy 22.86 111.76) (xy 22.86 114.3))
-    (stroke (width 0) (type default))
-  )
   (wire (pts (xy 144.145 44.45) (xy 167.64 44.45))
     (stroke (width 0) (type default))
@@
     (stroke (width 0) (type default))
   )
-  (wire (pts (xy 22.86 99.06) (xy 22.86 104.14))
-    (stroke (width 0) (type default))
-  )
   (wire (pts (xy 36.83 96.52) (xy 36.83 99.06))
     (stroke (width 0) (type default))
@@
     (stroke (width 0) (type default))
   )
+  (wire (pts (xy 81.28 97.79) (xy 81.28 102.87))
+    (stroke (width 0) (type default))
+  )
   (wire (pts (xy 132.715 44.45) (xy 144.145 44.45))
     (stroke (width 0) (type default))
@@
     (stroke (width 0) (type default))
   )
+  (wire (pts (xy 77.47 97.79) (xy 81.28 97.79))
+    (stroke (width 0) (type default))
+  )
   (wire (pts (xy 50.8 54.0004) (xy 50.8 55.88))
     (stroke (width 0) (type default))
   )
-  (wire (pts (xy 81.28 93.98) (xy 81.28 102.87))
+  (wire (pts (xy 81.28 93.98) (xy 81.28 97.79))
     (stroke (width 0) (type default))
   )
@@
     )
   )
-  (symbol (lib_id "power:GND") (at 22.86 114.3 0) (unit 1)
-    (in_bom yes) (on_board yes) (dnp no)
-    (property "Reference" "#PWR09" (at 22.86 120.65 0)
-      (effects (font (size 1.27 1.27)) hide)
-    )
-    (property "Value" "GND" (at 22.86 118.11 0)
-      (effects (font (size 1.27 1.27)))
-    )
-    (property "Footprint" "" (at 22.86 114.3 0)
-      (effects (font (size 1.27 1.27)) hide)
-    )
-    (property "Datasheet" "" (at 22.86 114.3 0)
+  (symbol (lib_id "power:GND") (at 69.85 97.79 0) (unit 1)
+    (in_bom yes) (on_board yes) (dnp no)
+    (property "Reference" "#PWR09" (at 69.85 104.14 0)
+      (effects (font (size 1.27 1.27)) hide)
+    )
+    (property "Value" "GND" (at 69.85 101.6 0)
+      (effects (font (size 1.27 1.27)))
+    )
+    (property "Footprint" "" (at 69.85 97.79 0)
+      (effects (font (size 1.27 1.27)) hide)
+    )
+    (property "Datasheet" "" (at 69.85 97.79 0)
       (effects (font (size 1.27 1.27)) hide)
     )
@@
     )
   )
-  (symbol (lib_id "Device:C") (at 22.86 107.95 0) (unit 1)
-    (in_bom yes) (on_board yes) (dnp no)
-    (property "Reference" "C17" (at 25.4 106.68 0)
-      (effects (font (size 1.27 1.27)) (justify left))
-    )
-    (property "Value" "1uF" (at 25.4 109.22 0)
-      (effects (font (size 1.27 1.27)) (justify left))
-    )
-    (property "Footprint" "Capacitor_SMD:C_0805_2012Metric" (at 23.8252 111.76 0)
-      (effects (font (size 1.27 1.27)) hide)
-    )
-    (property "Datasheet" "~" (at 22.86 107.95 0)
+  (symbol (lib_id "Device:C") (at 73.66 97.79 90) (unit 1)
+    (in_bom yes) (on_board yes) (dnp no)
+    (property "Reference" "C17" (at 76.2 93.98 90)
+      (effects (font (size 1.27 1.27)) (justify left))
+    )
+    (property "Value" "1uF" (at 76.2 101.6 90)
+      (effects (font (size 1.27 1.27)) (justify left))
+    )
+    (property "Footprint" "Capacitor_SMD:C_0805_2012Metric" (at 77.47 96.8248 0)
+      (effects (font (size 1.27 1.27)) hide)
+    )
+    (property "Datasheet" "~" (at 73.66 97.79 0)
       (effects (font (size 1.27 1.27)) hide)
     )
@@
         )
       )
-    )
-  )
-  (symbol (lib_id "power:+BATT") (at 22.86 99.06 0) (unit 1)
-    (in_bom yes) (on_board yes) (dnp no) (fields_autoplaced)
-    (property "Reference" "#PWR04" (at 22.86 102.87 0)
-      (effects (font (size 1.27 1.27)) hide)
-    )
-    (property "Value" "+BATT" (at 22.86 94.6912 0)
-      (effects (font (size 1.27 1.27)))
-    )
-    (property "Footprint" "" (at 22.86 99.06 0)
-      (effects (font (size 1.27 1.27)) hide)
-    )
-    (property "Datasheet" "" (at 22.86 99.06 0)
-      (effects (font (size 1.27 1.27)) hide)
-    )
-    (pin "1")
-    (instances
-      (project "MuscleRecoveryV1"
-        (path "/4e550305-79d2-4e4a-a502-817ebcc79f9a/648f095b-a230-48ff-8dbf-d0fbef398770"
-          (reference "#PWR04") (unit 1)
-        )
-      )
-      (project "Power For Muscle Recovery"
-        (path "/68ba6acb-d7b0-4091-ad4f-10769cda4f80"
-          (reference "#PWR02") (unit 1)
-        )
-      )
-      (project "New Test"
-        (path "/ec7ffed6-1d2d-48f7-b073-d0a7d4b8c858"
-          (reference "#PWR03") (unit 1)
-        )
-      )
