File: production/ecad/MuscleRecoveryV1/MuscleRecoveryV1.kicad_sch (KiCad schematic)
At the start: 17 parts, among them J3 Screw_Terminal_01x06, U6 ESP32-WROOM-32

Commit message: Display commit 1
Parts:
- removed 3v31, GND1, MISO1, MOSI1, SCL, SDA1, SD_CS1, TFT_CLK1, TFT_CS1, TFT_DC1, TFT_RST1: TestPoint, symbol Connector:TestPoint
- removed C12: 1uF, symbol Device:C_Small
- removed C13: 10uF, symbol Device:C_Small
- removed J3: Screw_Terminal_01x06, symbol Connector:Screw_Terminal_01x06
- removed R30, R31: 4.7k, symbol Device:R
- removed U6: ESP32-WROOM-32, RF_Module:ESP32-WROOM-32, symbol RF_Module:ESP32-WROOM-32
- added U4: ESP32-WROOM-32E-N8, symbol ESP32-WROOM-32E-N8:ESP32-WROOM-32E-N8
Connections:
- no-connect marks 15 -> 0
Other:
- sheet Bootloading ports: added none; removed EN, IO0, RXD0, TXD0
- sheet Display ports: added none; removed MISO, MOSI, SD_CS, TFT_CLK, TFT_CS, TFT_DC, TFT_RST
- sheet EMG ports: added none; removed ALERT/LABEL, SCL, SDA
- sheet Power and Battery ports: added none; removed SCL, SDA
