File: production/ecad/MuscleRecoveryV2 Copy/MuscleDisplay.kicad_sch (KiCad schematic)
At the start: 18 parts, among them J3 Motor_Screw_Terminal, J7 Conn_01x11_Pin, Q4 AO3400A

Commit message: Created New Layout
Parts:
- D7: footprint LED_THT:LED_D1.8mm_W3.3mm_H2.4mm -> LED_SMD:LED_0402_1005Metric
- J3: footprint (none) -> Connector_PinHeader_2.54mm:PinHeader_1x02_P2.54mm_Vertical
- J7: footprint (none) -> Connector_PinHeader_2.54mm:PinHeader_1x11_P2.54mm_Horizontal
- R35, R53, R54, R55, R56, R57, R58, R59, R60: footprint (none) -> Resistor_SMD:R_0402_1005Metric
- R50, R51, R52: footprint (none) -> Resistor_SMD:R_01005_0402Metric
- S1, S4: footprint B3F-1000:SW_B3F-1000 -> Muscle_Recovery_Footprint_Library:SW_B3F-1000
Changed lines of the file:
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@@
       (effects (font (size 1.27 1.27)))
     )
-    (property "Footprint" "" (at 123.19 41.91 0)
+    (property "Footprint" "Resistor_SMD:R_0402_1005Metric" (at 123.19 41.91 0)
       (effects (font (size 1.27 1.27)) hide)
     )
@@
       (effects (font (size 1.27 1.27)))
     )
-    (property "Footprint" "" (at 123.19 59.69 0)
+    (property "Footprint" "Resistor_SMD:R_0402_1005Metric" (at 123.19 59.69 0)
       (effects (font (size 1.27 1.27)) hide)
     )
@@
       (effects (font (size 1.27 1.27)))
     )
-    (property "Footprint" "" (at 123.19 52.07 0)
+    (property "Footprint" "Resistor_SMD:R_0402_1005Metric" (at 123.19 52.07 0)
       (effects (font (size 1.27 1.27)) hide)
     )
@@
       (effects (font (size 1.27 1.27)))
     )
-    (property "Footprint" "LED_THT:LED_D1.8mm_W3.3mm_H2.4mm" (at 181.61 96.52 90)
+    (property "Footprint" "LED_SMD:LED_0402_1005Metric" (at 181.61 96.52 90)
       (effects (font (size 1.27 1.27)) hide)
     )
@@
       (effects (font (size 1.27 1.27)))
     )
-    (property "Footprint" "" (at 123.19 49.53 0)
+    (property "Footprint" "Resistor_SMD:R_01005_0402Metric" (at 123.19 49.53 0)
       (effects (font (size 1.27 1.27)) hide)
     )
@@
       (effects (font (size 1.27 1.27)) (justify left))
     )
-    (property "Footprint" "" (at 172.72 95.25 0)
+    (property "Footprint" "Connector_PinHeader_2.54mm:PinHeader_1x02_P2.54mm_Vertical" (at 172.72 95.25 0)
       (effects (font (size 1.27 1.27)) hide)
     )
@@
       (effects (font (size 1.27 1.27)))
     )
-    (property "Footprint" "" (at 123.19 54.61 0)
+    (property "Footprint" "Resistor_SMD:R_0402_1005Metric" (at 123.19 54.61 0)
       (effects (font (size 1.27 1.27)) hide)
     )
@@
       (effects (font (size 1.27 1.27)))
     )
-    (property "Footprint" "" (at 123.19 44.45 0)
+    (property "Footprint" "Resistor_SMD:R_01005_0402Metric" (at 123.19 44.45 0)
       (effects (font (size 1.27 1.27)) hide)
     )
@@
       (effects (font (size 1.27 1.27)))
     )
-    (property "Footprint" "" (at 137.16 46.99 0)
+    (property "Footprint" "Connector_PinHeader_2.54mm:PinHeader_1x11_P2.54mm_Horizontal" (at 137.16 46.99 0)
       (effects (font (size 1.27 1.27)) hide)
     )
@@
       (effects (font (size 1.27 1.27)) (justify left))
     )
-    (property "Footprint" "" (at 60.96 137.16 0)
+    (property "Footprint" "Resistor_SMD:R_0402_1005Metric" (at 60.96 137.16 0)
       (effects (font (size 1.27 1.27)) hide)
     )
@@
       (effects (font (size 1.27 1.27)) (justify left))
     )
-    (property "Footprint" "" (at 60.96 92.71 0)
+    (property "Footprint" "Resistor_SMD:R_0402_1005Metric" (at 60.96 92.71 0)
       (effects (font (size 1.27 1.27)) hide)
     )
@@
       (effects (font (size 1.27 1.27)))
     )
-    (property "Footprint" "B3F-1000:SW_B3F-1000" (at 76.2 109.22 0)
+    (property "Footprint" "Muscle_Recovery_Footprint_Library:SW_B3F-1000" (at 76.2 109.22 0)
       (effects (font (size 1.27 1.27)) (justify bottom) hide)
     )
@@
       (effects (font (size 1.27 1.27)))
     )
-    (property "Footprint" "" (at 123.19 46.99 0)
+    (property "Footprint" "Resistor_SMD:R_01005_0402Metric" (at 123.19 46.99 0)
       (effects (font (size 1.27 1.27)) hide)
     )
@@
       (effects (font (size 1.27 1.27)))
     )
-    (property "Footprint" "B3F-1000:SW_B3F-1000" (at 76.2 153.67 0)
+    (property "Footprint" "Muscle_Recovery_Footprint_Library:SW_B3F-1000" (at 76.2 153.67 0)
       (effects (font (size 1.27 1.27)) (justify bottom) hide)
     )
@@
       (effects (font (size 1.27 1.27)))
     )
-    (property "Footprint" "" (at 149.86 113.03 0)
+    (property "Footprint" "Resistor_SMD:R_0402_1005Metric" (at 149.86 113.03 0)
       (effects (font (size 1.27 1.27)) hide)
     )
@@
       (effects (font (size 1.27 1.27)))
     )
-    (property "Footprint" "" (at 123.19 57.15 0)
+    (property "Footprint" "Resistor_SMD:R_0402_1005Metric" (at 123.19 57.15 0)
       (effects (font (size 1.27 1.27)) hide)
     )
@@
       (effects (font (size 1.27 1.27)) (justify left))
     )
-    (property "Footprint" "" (at 158.75 118.11 0)
-      (effects (font (size 1.27 1.27)) hide)
-    )
+    (property "Footprint" "Resistor_SMD:R_0402_1005Metric" (at 158.75 118.11 0)
+      (effects (font (size 1.27 1.27)) hide)
+    )

Commit message: Pushing Layout Changes for Andy's Layout
Parts:
- R50, R51, R52: footprint Resistor_SMD:R_01005_0402Metric -> Resistor_SMD:R_0402_1005Metric
- S1, S4: footprint Muscle_Recovery_Footprint_Library:SW_B3F-1000 -> Muscle_Recovery_Footprint_Library:PTS810SJG250SMTRLFS
Changed lines of the file:
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@@
       (effects (font (size 1.27 1.27)))
     )
-    (property "Footprint" "Resistor_SMD:R_01005_0402Metric" (at 123.19 49.53 0)
+    (property "Footprint" "Resistor_SMD:R_0402_1005Metric" (at 123.19 49.53 0)
       (effects (font (size 1.27 1.27)) hide)
     )
@@
       (effects (font (size 1.27 1.27)))
     )
-    (property "Footprint" "Resistor_SMD:R_01005_0402Metric" (at 123.19 44.45 0)
+    (property "Footprint" "Resistor_SMD:R_0402_1005Metric" (at 123.19 44.45 0)
       (effects (font (size 1.27 1.27)) hide)
     )
@@
       (effects (font (size 1.27 1.27)))
     )
-    (property "Footprint" "Muscle_Recovery_Footprint_Library:SW_B3F-1000" (at 76.2 109.22 0)
+    (property "Footprint" "Muscle_Recovery_Footprint_Library:PTS810SJG250SMTRLFS" (at 76.2 109.22 0)
       (effects (font (size 1.27 1.27)) (justify bottom) hide)
     )
@@
       (effects (font (size 1.27 1.27)))
     )
-    (property "Footprint" "Resistor_SMD:R_01005_0402Metric" (at 123.19 46.99 0)
+    (property "Footprint" "Resistor_SMD:R_0402_1005Metric" (at 123.19 46.99 0)
       (effects (font (size 1.27 1.27)) hide)
     )
@@
       (effects (font (size 1.27 1.27)))
     )
-    (property "Footprint" "Muscle_Recovery_Footprint_Library:SW_B3F-1000" (at 76.2 153.67 0)
-      (effects (font (size 1.27 1.27)) (justify bottom) hide)
-    )
+    (property "Footprint" "Muscle_Recovery_Footprint_Library:PTS810SJG250SMTRLFS" (at 76.2 153.67 0)
+      (effects (font (size 1.27 1.27)) (justify bottom) hide)
+    )

Commit message: Committing My pliminary placement for my PCB <3
Parts:
- removed J7: Conn_01x11_Pin, Connector_PinHeader_2.54mm:PinHeader_1x11_P2.54mm_Horizontal, symbol Connector:Conn_01x11_Pin
- removed R35, R50, R51, R52, R53, R54, R55, R56: 0, Resistor_SMD:R_0402_1005Metric, symbol Device:R_Small
- removed S1, S4: B3F-1000, Muscle_Recovery_Footprint_Library:PTS810SJG250SMTRLFS, symbol B3F-1000:B3F-1000
- added J7: 51296-1894, Muscle_Recovery_Footprint_Library:512961894, symbol MuscleRecoverySymbolLibray:51296-1894
- added S1, S5: TL1105VF160Q, Muscle_Recovery_Footprint_Library:SW_TL1105VF160Q, symbol MuscleRecoverySymbolLibray:TL1105VF160Q
Connections:
- net +3.3V: now also J7.1, S1.2, S5.2
- net ALT_START_BUTTON: now also S1.1
- net GND: now also J7.2
- net LIT: now also J7.10
- net MISO: now also J7.4
- net MOSI: now also J7.5
- net SCK: now also J7.3
- net SD_CS: now also J7.9
- net START_BUTTON: now also S5.1
- net TFT_CS: now also J7.6
- net TFT_DC: now also J7.8
- net TFT_RST: now also J7.7
- no-connect marks 5 -> 11
Other:
- note removed: "TFT SCREEN CONNECTOR *include SPI bus for SD Card & TFT screen - SCK - miso (only for SD card) - mosi - SD_CS & TFT_CS"

Commit message: Adding additional components to library for final rev2 changes
Parts:
- added H1, H2, H3, H4: MountingHole, Muscle_Recovery_Footprint_Library:MH, symbol Mechanical:MountingHole
Other:
- note added: "Mounting Holes"
Changed lines of the file:
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@@
     (fill (type none))
   )
-  (rectangle (start 91.44 20.32) (end 186.69 64.77)
+  (rectangle (start 34.925 20.955) (end 130.175 65.405)
     (stroke (width 0) (type default))
     (fill (type none))
   )
   (text "Vibration motor control\n" (at 189.23 132.08 0)
+    (effects (font (size 1.27 1.27)) (justify left bottom))
+  )
+  (text "Mounting Holes" (at 36.195 24.13 0)
     (effects (font (size 1.27 1.27)) (justify left bottom))
   )
@@
     )
   )
+  (symbol (lib_id "Mechanical:MountingHole") (at 108.585 36.83 0) (unit 1)
+    (in_bom yes) (on_board yes) (dnp no) (fields_autoplaced)
+    (property "Reference" "H4" (at 111.125 35.56 0)
+      (effects (font (size 1.27 1.27)) (justify left))
+    )
+    (property "Value" "MountingHole" (at 111.125 38.1 0)
+      (effects (font (size 1.27 1.27)) (justify left))
+    )
+    (property "Footprint" "Muscle_Recovery_Footprint_Library:MH" (at 108.585 36.83 0)
+      (effects (font (size 1.27 1.27)) hide)
+    )
+    (property "Datasheet" "~" (at 108.585 36.83 0)
+      (effects (font (size 1.27 1.27)) hide)
+    )
+    (instances
+      (project "MuscleRecoveryV1"
+        (path "/4e550305-79d2-4e4a-a502-817ebcc79f9a/85edd68f-6119-4dbf-9af0-99f996378c09"
+          (reference "H4") (unit 1)
+        )
+      )
+    )
+  )
   (symbol (lib_id "Connector:Screw_Terminal_01x02") (at 172.72 95.25 0) (unit 1)
     (in_bom yes) (on_board yes) (dnp no)
@@
         (path "/4e550305-79d2-4e4a-a502-817ebcc79f9a/85edd68f-6119-4dbf-9af0-99f996378c09"
           (reference "J3") (unit 1)
+        )
+      )
+    )
+  )
+  (symbol (lib_id "Mechanical:MountingHole") (at 68.58 36.83 0) (unit 1)
+    (in_bom yes) (on_board yes) (dnp no) (fields_autoplaced)
+    (property "Reference" "H2" (at 71.12 35.56 0)
+      (effects (font (size 1.27 1.27)) (justify left))
+    )
+    (property "Value" "MountingHole" (at 71.12 38.1 0)
+      (effects (font (size 1.27 1.27)) (justify left))
+    )
+    (property "Footprint" "Muscle_Recovery_Footprint_Library:MH" (at 68.58 36.83 0)
+      (effects (font (size 1.27 1.27)) hide)
+    )
+    (property "Datasheet" "~" (at 68.58 36.83 0)
+      (effects (font (size 1.27 1.27)) hide)
+    )
+    (instances
+      (project "MuscleRecoveryV1"
+        (path "/4e550305-79d2-4e4a-a502-817ebcc79f9a/85edd68f-6119-4dbf-9af0-99f996378c09"
+          (reference "H2") (unit 1)
+        )
+      )
+    )
+  )
+  (symbol (lib_id "Mechanical:MountingHole") (at 88.9 36.83 0) (unit 1)
+    (in_bom yes) (on_board yes) (dnp no) (fields_autoplaced)
+    (property "Reference" "H3" (at 91.44 35.56 0)
+      (effects (font (size 1.27 1.27)) (justify left))
+    )
+    (property "Value" "MountingHole" (at 91.44 38.1 0)
+      (effects (font (size 1.27 1.27)) (justify left))
+    )
+    (property "Footprint" "Muscle_Recovery_Footprint_Library:MH" (at 88.9 36.83 0)
+      (effects (font (size 1.27 1.27)) hide)
+    )
+    (property "Datasheet" "~" (at 88.9 36.83 0)
+      (effects (font (size 1.27 1.27)) hide)
+    )
+    (instances
+      (project "MuscleRecoveryV1"
+        (path "/4e550305-79d2-4e4a-a502-817ebcc79f9a/85edd68f-6119-4dbf-9af0-99f996378c09"
+          (reference "H3") (unit 1)
         )
       )
@@
         )
       )
+    )
+  )
+  (symbol (lib_id "Mechanical:MountingHole") (at 48.26 36.83 0) (unit 1)
+    (in_bom yes) (on_board yes) (dnp no) (fields_autoplaced)
+    (property "Reference" "H1" (at 50.8 35.56 0)
+      (effects (font (size 1.27 1.27)) (justify left))
+    )
+    (property "Value" "MountingHole" (at 50.8 38.1 0)
+      (effects (font (size 1.27 1.27)) (justify left))
+    )
+    (property "Footprint" "Muscle_Recovery_Footprint_Library:MH" (at 48.26 36.83 0)
+      (effects (font (size 1.27 1.27)) hide)
+    )
+    (property "Datasheet" "~" (at 48.26 36.83 0)
+      (effects (font (size 1.27 1.27)) hide)
+    )
+    (instances
+      (project "MuscleRecoveryV1"
+        (path "/4e550305-79d2-4e4a-a502-817ebcc79f9a/85edd68f-6119-4dbf-9af0-99f996378c09"
+          (reference "H1") (unit 1)
+        )
+      )

Commit message: committing some recent changes to layout
Parts:
- removed R57: 10k, Resistor_SMD:R_0402_1005Metric, symbol Device:R_Small
- removed S1, S5: TL1105VF160Q, Muscle_Recovery_Footprint_Library:SW_TL1105VF160Q, symbol MuscleRecoverySymbolLibray:TL1105VF160Q
- added J2, J8: SM02B-SRSS-TB_LF__SN_, Muscle_Recovery_Footprint_Library:SM02B-SRSS-TB_LF__SN_, symbol MuscleRecoverySymbolLibray:SM02B-SRSS-TB_LF__SN_
- added R51: 10k, Resistor_SMD:R_0402_1005Metric, symbol Device:R_Small
- H1, H2, H3, H4: footprint Muscle_Recovery_Footprint_Library:MH -> MountingHole:MountingHole_3.2mm_M3
- J3: footprint Connector_PinHeader_2.54mm:PinHeader_1x02_P2.54mm_Vertical -> Muscle_Recovery_Footprint_Library:Motor_Conn
Connections:
- net +3.3V: now also J2.1, J8.1
- net ALT_START_BUTTON: now also J2.2
- net GND: now also J7.3, R51.2; no longer J7.2
- net LIT: now also J7.2; no longer J7.10
- net MISO: now also J7.6; no longer J7.4
- net SCK: now also J7.4; no longer J7.3
- net SD_CS: now also J7.10; no longer J7.9
- net START_BUTTON: now also J8.2, R51.1
- net TFT_CS: now also J7.8; no longer J7.6
- net TFT_DC: now also J7.7; no longer J7.8
- net TFT_RST: now also J7.9; no longer J7.7
- no-connect marks 11 -> 12
Other:
- note added: "M3 Mounting Holes"
- moved on the sheet: D7, J3, Q4, R58, R59, R60

Commit message: Pushing Most of the final changes for PCB REV2
Parts:
- removed D7: LED_Small, LED_SMD:LED_0402_1005Metric, symbol Device:LED_Small
- removed J2: SM02B-SRSS-TB_LF__SN_, Muscle_Recovery_Footprint_Library:SM02B-SRSS-TB_LF__SN_, symbol MuscleRecoverySymbolLibray:SM02B-SRSS-TB_LF__SN_
- removed J3: Motor_Screw_Terminal, Muscle_Recovery_Footprint_Library:Motor_Conn, symbol Connector:Screw_Terminal_01x02
- removed Q4: AO3400A, Package_TO_SOT_SMD:SOT-23, symbol Transistor_FET:AO3400A
- removed R58: 10k, Resistor_SMD:R_0402_1005Metric, symbol Device:R_Small
- added D7: 1N914WT, Diode_SMD:D_SOD-523, symbol Diode:1N914WT
- added J3, J4: SM02B-SRSS-TB_LF__SN_, Muscle_Recovery_Footprint_Library:SM02B-SRSS-TB_LF__SN_, symbol MuscleRecoverySymbolLibray:SM02B-SRSS-TB_LF__SN_
- added Q2: AO3400A, Package_TO_SOT_SMD:SOT-23, symbol Transistor_FET:AO3400A
- added R29: 10k, Resistor_SMD:R_0402_1005Metric, symbol Device:R_Small
Connections:
- net ALT_START_BUTTON: now also J4.2, R29.1
- net GND: now also J7.16, Q2.2 (S), R29.2; no longer J7.3
- net LIT: now also J7.17; no longer J7.2
- net MISO: now also J7.13; no longer J7.6
- net MOSI: now also J7.14; no longer J7.5
- net SCK: now also J7.15; no longer J7.4
- net SD_CS: now also J7.9; no longer J7.10
- net TFT_CS: now also J7.11; no longer J7.8
- net TFT_DC: now also J7.12; no longer J7.7
- net TFT_RST: now also J7.10; no longer J7.9
- net +3V3: now reaches J7.18
- net +3V3: now also J8.1, D7.1 (K), J3.1, J4.1
- net at R59.1, R60.2: now also Q2.1 (G)
- net +3.3V: no longer names the net of J7.1
- net +3.3V: no longer J8.1
- new net: D7.2 (A), J3.2, Q2.3 (D)
- no-connect marks 12 -> 10
Other:
- moved on the sheet: J7
