File: production/ecad/MuscleRecoveryV2 Copy/MuscleBooting.kicad_sch (KiCad schematic)
At the start: 25 parts, among them J4 USB_C_Receptacle_USB2.0, Q2 AO3400A, Q3 AO3400A, U3 CP2102N-Axx-xQFN28

Commit message: Created New Layout
Parts:
- C6, C7, C8, C9: footprint Capacitor_SMD:C_0805_2012Metric -> Capacitor_SMD:C_0402_1005Metric
- R10, R11, R12, R13, R14, R15, R16, R17, R18, R40, R8, R9: footprint Resistor_SMD:R_0805_2012Metric -> Resistor_SMD:R_0402_1005Metric
- S2, S3: footprint B3F-1000:SW_B3F-1000 -> Muscle_Recovery_Footprint_Library:SW_B3F-1000
Changed lines of the file:
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@@
       (effects (font (size 1.27 1.27)))
     )
-    (property "Footprint" "Resistor_SMD:R_0805_2012Metric" (at 40.8432 138.303 0)
+    (property "Footprint" "Resistor_SMD:R_0402_1005Metric" (at 40.8432 138.303 0)
       (effects (font (size 1.27 1.27)) hide)
     )
@@
       (effects (font (size 1.27 1.27)))
     )
-    (property "Footprint" "B3F-1000:SW_B3F-1000" (at 115.57 154.94 0)
+    (property "Footprint" "Muscle_Recovery_Footprint_Library:SW_B3F-1000" (at 115.57 154.94 0)
       (effects (font (size 1.27 1.27)) (justify bottom) hide)
     )
@@
       (effects (font (size 1.27 1.27)) (justify left))
     )
-    (property "Footprint" "Resistor_SMD:R_0805_2012Metric" (at 141.859 118.11 0)
+    (property "Footprint" "Resistor_SMD:R_0402_1005Metric" (at 141.859 118.11 0)
       (effects (font (size 1.27 1.27)) hide)
     )
@@
       (effects (font (size 1.27 1.27)))
     )
-    (property "Footprint" "Resistor_SMD:R_0805_2012Metric" (at 40.64 122.555 0)
+    (property "Footprint" "Resistor_SMD:R_0402_1005Metric" (at 40.64 122.555 0)
       (effects (font (size 1.27 1.27)) hide)
     )
@@
       (effects (font (size 1.27 1.27)))
     )
-    (property "Footprint" "Resistor_SMD:R_0805_2012Metric" (at 175.641 126.492 0)
+    (property "Footprint" "Resistor_SMD:R_0402_1005Metric" (at 175.641 126.492 0)
       (effects (font (size 1.27 1.27)) hide)
     )
@@
       (effects (font (size 1.27 1.27)) (justify left))
     )
-    (property "Footprint" "Resistor_SMD:R_0805_2012Metric" (at 147.701 67.691 0)
+    (property "Footprint" "Resistor_SMD:R_0402_1005Metric" (at 147.701 67.691 0)
       (effects (font (size 1.27 1.27)) hide)
     )
@@
       (effects (font (size 1.27 1.27)) (justify left))
     )
-    (property "Footprint" "Capacitor_SMD:C_0805_2012Metric" (at 139.446 51.435 0)
+    (property "Footprint" "Capacitor_SMD:C_0402_1005Metric" (at 139.446 51.435 0)
       (effects (font (size 1.27 1.27)) hide)
     )
@@
       (effects (font (size 1.27 1.27)) (justify left))
     )
-    (property "Footprint" "Resistor_SMD:R_0805_2012Metric" (at 147.701 74.295 0)
+    (property "Footprint" "Resistor_SMD:R_0402_1005Metric" (at 147.701 74.295 0)
       (effects (font (size 1.27 1.27)) hide)
     )
@@
       (effects (font (size 1.27 1.27)) (justify left))
     )
-    (property "Footprint" "Resistor_SMD:R_0805_2012Metric" (at 74.041 70.485 0)
+    (property "Footprint" "Resistor_SMD:R_0402_1005Metric" (at 74.041 70.485 0)
       (effects (font (size 1.27 1.27)) hide)
     )
@@
       (effects (font (size 1.27 1.27)) (justify left))
     )
-    (property "Footprint" "Capacitor_SMD:C_0805_2012Metric" (at 126.365 128.397 0)
+    (property "Footprint" "Capacitor_SMD:C_0402_1005Metric" (at 126.365 128.397 0)
       (effects (font (size 1.27 1.27)) hide)
     )
@@
       (effects (font (size 1.27 1.27)) (justify left))
     )
-    (property "Footprint" "Resistor_SMD:R_0805_2012Metric" (at 168.783 66.548 0)
+    (property "Footprint" "Resistor_SMD:R_0402_1005Metric" (at 168.783 66.548 0)
       (effects (font (size 1.27 1.27)) hide)
     )
@@
       (effects (font (size 1.27 1.27)) (justify left))
     )
-    (property "Footprint" "Capacitor_SMD:C_0805_2012Metric" (at 86.106 129.413 0)
+    (property "Footprint" "Capacitor_SMD:C_0402_1005Metric" (at 86.106 129.413 0)
       (effects (font (size 1.27 1.27)) hide)
     )
@@
       (effects (font (size 1.27 1.27)))
     )
-    (property "Footprint" "Resistor_SMD:R_0805_2012Metric" (at 175.641 135.128 0)
+    (property "Footprint" "Resistor_SMD:R_0402_1005Metric" (at 175.641 135.128 0)
       (effects (font (size 1.27 1.27)) hide)
     )
@@
       (effects (font (size 1.27 1.27)))
     )
-    (property "Footprint" "B3F-1000:SW_B3F-1000" (at 155.829 153.543 0)
+    (property "Footprint" "Muscle_Recovery_Footprint_Library:SW_B3F-1000" (at 155.829 153.543 0)
       (effects (font (size 1.27 1.27)) (justify bottom) hide)
     )
@@
       (effects (font (size 1.27 1.27)) (justify left))
     )
-    (property "Footprint" "Capacitor_SMD:C_0805_2012Metric" (at 152.4 51.435 0)
+    (property "Footprint" "Capacitor_SMD:C_0402_1005Metric" (at 152.4 51.435 0)
       (effects (font (size 1.27 1.27)) hide)
     )
@@
       (effects (font (size 1.27 1.27)) (justify left))
     )
-    (property "Footprint" "Resistor_SMD:R_0805_2012Metric" (at 60.071 70.612 0)
+    (property "Footprint" "Resistor_SMD:R_0402_1005Metric" (at 60.071 70.612 0)
       (effects (font (size 1.27 1.27)) hide)
     )
@@
       (effects (font (size 1.27 1.27)) (justify left))
     )
-    (property "Footprint" "Resistor_SMD:R_0805_2012Metric" (at 101.6 119.126 0)
+    (property "Footprint" "Resistor_SMD:R_0402_1005Metric" (at 101.6 119.126 0)
       (effects (font (size 1.27 1.27)) hide)
     )
@@
       (effects (font (size 1.27 1.27)) (justify left))
     )
-    (property "Footprint" "Resistor_SMD:R_0805_2012Metric" (at 172.593 33.528 0)
-      (effects (font (size 1.27 1.27)) hide)
-    )
+    (property "Footprint" "Resistor_SMD:R_0402_1005Metric" (at 172.593 33.528 0)
+      (effects (font (size 1.27 1.27)) hide)
+    )

Commit message: Pushing Layout Changes for Andy's Layout
Parts:
- S2, S3: footprint Muscle_Recovery_Footprint_Library:SW_B3F-1000 -> Muscle_Recovery_Footprint_Library:PTS810SJG250SMTRLFS
Changed lines of the file:
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@@
       (effects (font (size 1.27 1.27)))
     )
-    (property "Footprint" "Muscle_Recovery_Footprint_Library:SW_B3F-1000" (at 115.57 154.94 0)
+    (property "Footprint" "Muscle_Recovery_Footprint_Library:PTS810SJG250SMTRLFS" (at 115.57 154.94 0)
       (effects (font (size 1.27 1.27)) (justify bottom) hide)
     )
@@
       (effects (font (size 1.27 1.27)))
     )
-    (property "Footprint" "Muscle_Recovery_Footprint_Library:SW_B3F-1000" (at 155.829 153.543 0)
-      (effects (font (size 1.27 1.27)) (justify bottom) hide)
-    )
+    (property "Footprint" "Muscle_Recovery_Footprint_Library:PTS810SJG250SMTRLFS" (at 155.829 153.543 0)
+      (effects (font (size 1.27 1.27)) (justify bottom) hide)
+    )

Commit message: Committing My pliminary placement for my PCB <3
Connections:
- no-connect marks 22 -> 23
Changed lines of the file:
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@@
   (no_connect (at 208.915 54.737))
   (no_connect (at 208.915 50.927))
+  (no_connect (at 203.835 36.195))
   (no_connect (at 177.165 68.707))
   (no_connect (at 159.639 129.413))

Commit message: Adding more updates to Rev2 Layout
Parts:
- added BT1: 3034, Muscle_Recovery_Footprint_Library:BAT_3034, symbol MuscleRecoverySymbolLibray:3034
- added IC2: W25Q128JVPIQ, Muscle_Recovery_Footprint_Library:SON127P600X500X80-9N-D, symbol MuscleRecoverySymbolLibray:W25Q128JVPIQ
- added LS1: PKLCS1212E4001-R1, Muscle_Recovery_Footprint_Library:SPKR_PKLCS1212E4001-R1, symbol MuscleRecoverySymbolLibray:PKLCS1212E4001-R1
- added U4: PCF8523T/1_118, Muscle_Recovery_Footprint_Library:SO8_SOT96-1_NXP, symbol MuscleRecoverySymbolLibray:PCF8523T_1_118
Other:
- note added: "RTC"
- note added: "SPI Flash"
- note added: "Speaker"

Commit message: committing some recent changes to layout
Parts:
- removed BT1: 3034, Muscle_Recovery_Footprint_Library:BAT_3034, symbol MuscleRecoverySymbolLibray:3034
- added C19, C22, C23: 1uF, Capacitor_SMD:C_0402_1005Metric, symbol Device:C_Small
- added C20, C21: 10pF, Capacitor_SMD:C_0402_1005Metric, symbol Device:C_Small
- added R27, R35, R50: 10K, Resistor_SMD:R_0402_1005Metric, symbol Device:R_Small
- added Y1: ABS07-32.768KHZ-7-T, Muscle_Recovery_Footprint_Library:XTAL_ABS07-32.768KHZ-7-T, symbol MuscleRecoverySymbolLibray:ABS07-32.768KHZ-7-T
- J4: footprint Connector_USB:USB_C_Plug_Molex_105444 -> Muscle_Recovery_Footprint_Library:USB4110-GF-A_GCT
Connections:
- net +3.3V: now also IC2.8 (VCC), U4.8 (VDD), C19.1, C22.1, R27.1, R35.1, R50.1
- net GND: now also IC2.4 (GND_1), IC2.9 (GND_2), LS1.N, U4.4 (VSS), C19.2, C20.2, C21.2, C22.2, C23.2
- net OSC1: now reaches U4.1 (OSCI)
- net OSC1: now also C20.1, Y1.1
- net OSC2: now reaches U4.2 (OSCO)
- net OSC2: now also C21.1, Y1.2
- net +BATT: now reaches U4.3 (VBAT)
- net +BATT: now also C23.1
- net SDA: now reaches U4.5 (SDA)
- net SCL: now reaches U4.6 (SCL)
- net SPI_CS_FLSH: now reaches IC2.1 (~{CS})
- net SPI_CS_FLSH: now also R27.2
- net MISO: now reaches IC2.2 (DO_(IO1))
- net MISO: now also IC2.5 (DI_(IO0))
- net at IC2.3 (~{WP_(IO2)}): now also R35.2
- net SCK: now reaches IC2.6 (CLK)
- net at IC2.7 (~{HOLD_OR_}/RESET_(IO3)): now also R50.2
- net SPKR: now reaches LS1.P
- no-connect marks 23 -> 24
Other:
- note added: "32.768 Crystal"
- moved on the sheet: IC2, LS1, U4

Commit message: Pushing Most of the final changes for PCB REV2
Parts:
- removed C6, C7: C_Small, Capacitor_SMD:C_0402_1005Metric, symbol Device:C_Small
- removed IO0, TP4, VBUS1: TestPoint, TestPoint:TestPoint_Pad_D1.5mm, symbol Connector:TestPoint
- removed J4: USB_C_Receptacle_USB2.0, Muscle_Recovery_Footprint_Library:USB4110-GF-A_GCT, symbol Connector:USB_C_Receptacle_USB2.0
- removed LS1: PKLCS1212E4001-R1, Muscle_Recovery_Footprint_Library:SPKR_PKLCS1212E4001-R1, symbol MuscleRecoverySymbolLibray:PKLCS1212E4001-R1
- removed S2, S3: B3F-1000, Muscle_Recovery_Footprint_Library:PTS810SJG250SMTRLFS, symbol B3F-1000:B3F-1000
- added C20: 1uF, Capacitor_SMD:C_0402_1005Metric, symbol Device:C_Small
- added C21: 0.1uF, Capacitor_SMD:C_0402_1005Metric, symbol Device:C_Small
- added J5: USB4110-GF-A, Muscle_Recovery_Footprint_Library:USB4110-GF-A_GCT, symbol MuscleRecoverySymbolLibray:USB4110-GF-A
- added U4: ADXL343, Package_LGA:LGA-14_3x5mm_P0.8mm_LayoutBorder1x6y, symbol Sensor_Motion:ADXL343
Connections:
- net GND: now also C20.2, C21.2, J5.A1-B12 (GND), J5.A12-B1 (GND), U4.2 (GND), U4.4 (GND), U4.5 (GND)
- net MISO: no longer IC2.5 (DI_(IO0))
- net SCL: now also U4.14 (SCL/SCLK)
- net SDA: now also U4.13 (SDA/SDI/SDIO)
- net USB+: now also J5.A7 (DN1), J5.B7 (DN2)
- net USB-: now also J5.A6 (DP1), J5.B6 (DP2)
- net VBUS: now also J5.A4-B9 (VBUS), J5.A9-B4 (VBUS)
- net at R10.1: now also J5.A5 (CC1)
- net at R9.1: now also J5.B5 (CC2)
- net +3.3V renamed +3V3
- net +3V3: now also C20.1, C21.1, U4.1 (Vdd_I/O), U4.12 (SDO/ADDR), U4.6 (Vs)
- new net MOSI: IC2.5 (DI_(IO0))
- no-connect marks 24 -> 26
Other:
- note added: "Accelerometer"
- note added: "NOTE: There are typically buttons here used for manual booting In this case, there is not a need for them since the manual boot circuit takes care of this. They have also been left off for form factor reasons"
- note removed: "DNI"

Commit message: Pushing changes post schematic review
Connections:
- net +3V3: now also U4.7 (~{CS})
- no-connect marks 26 -> 24
Other:
- note added: "0x1D"
Changed lines of the file:
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@@
   (junction (at 35.56 122.555) (diameter 0) (color 0 0 0 0)
+  )
+  (junction (at 237.49 203.2) (diameter 0) (color 0 0 0 0)
   )
   (junction (at 24.765 189.865) (diameter 0) (color 0 0 0 0)
@@
   (no_connect (at 208.915 50.927))
   (no_connect (at 266.065 208.28))
-  (no_connect (at 203.835 36.195))
   (no_connect (at 266.065 205.74))
   (no_connect (at 248.285 193.04))
@@
   (no_connect (at 208.915 63.627))
   (no_connect (at 258.445 218.44))
-  (no_connect (at 240.665 210.82))
   (wire (pts (xy 81.915 179.07) (xy 81.915 181.61))
     (stroke (width 0) (type default))
@@
     (stroke (width 0) (type default))
   )
+  (wire (pts (xy 240.665 210.82) (xy 237.49 210.82))
+    (stroke (width 0) (type default))
+  )
   (wire (pts (xy 238.76 154.94) (xy 252.73 154.94))
     (stroke (width 0) (type default))
   )
+  (wire (pts (xy 237.49 210.82) (xy 237.49 203.2))
+    (stroke (width 0) (type default))
+  )
   (wire (pts (xy 49.784 127.635) (xy 61.214 127.635))
     (stroke (width 0) (type default))
@@
     (stroke (width 0) (type default))
   )
-  (wire (pts (xy 235.585 203.2) (xy 240.665 203.2))
+  (wire (pts (xy 220.98 203.2) (xy 237.49 203.2))
     (stroke (width 0) (type default))
   )
@@
     (stroke (width 0) (type default))
   )
+  (wire (pts (xy 237.49 203.2) (xy 240.665 203.2))
+    (stroke (width 0) (type default))
+  )
   (wire (pts (xy 253.365 218.44) (xy 253.365 220.345))
     (stroke (width 0) (type default))
@@
     (stroke (width 0) (type default))
     (fill (type none))
+  )
+  (text "0x1D\n" (at 210.82 186.055 0)
+    (effects (font (size 1.27 1.27)) (justify left bottom))
   )
   (text "RTC" (at 125.73 167.64 0)
@@
     )
   )
-  (symbol (lib_id "power:+3V3") (at 235.585 203.2 0) (unit 1)
-    (in_bom yes) (on_board yes) (dnp no) (fields_autoplaced)
-    (property "Reference" "#PWR073" (at 235.585 207.01 0)
-      (effects (font (size 1.27 1.27)) hide)
-    )
-    (property "Value" "+3V3" (at 235.585 198.12 0)
-      (effects (font (size 1.27 1.27)))
-    )
-    (property "Footprint" "" (at 235.585 203.2 0)
-      (effects (font (size 1.27 1.27)) hide)
-    )
-    (property "Datasheet" "" (at 235.585 203.2 0)
-      (effects (font (size 1.27 1.27)) hide)
-    )
+  (symbol (lib_id "power:+3V3") (at 220.98 203.2 0) (unit 1)
+    (in_bom yes) (on_board yes) (dnp no) (fields_autoplaced)
+    (property "Reference" "#PWR073" (at 220.98 207.01 0)
+      (effects (font (size 1.27 1.27)) hide)
+    )
+    (property "Value" "+3V3" (at 220.98 198.12 0)
+      (effects (font (size 1.27 1.27)))
+    )
+    (property "Footprint" "" (at 220.98 203.2 0)
+      (effects (font (size 1.27 1.27)) hide)
+    )
+    (property "Datasheet" "" (at 220.98 203.2 0)
+      (effects (font (size 1.27 1.27)) hide)
+    )
