File: production/ecad/MuscleRecoveryV2 Copy/MuscleBooting.kicad_sch (KiCad schematic)
At the start: 32 parts, among them IC2 W25Q128JVPIQ, J5 USB4110-GF-A, Q2 AO3400A, Q3 AO3400A, U3 CP2102N-Axx-xQFN28, U4 ADXL343, U4 PCF8523T/1_118, Y1 ABS07-32.768KHZ-7-T

Commit message: Final Final FInal PCB
Parts:
- renumbered IC2 to U10
Changed lines of the file:
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@@
   (symbol (lib_id "MuscleRecoverySymbolLibray:W25Q128JVPIQ") (at 38.1 189.865 0) (unit 1)
     (in_bom yes) (on_board yes) (dnp no) (fields_autoplaced)
-    (property "Reference" "IC2" (at 44.45 183.515 0)
+    (property "Reference" "U10" (at 44.45 183.515 0)
       (effects (font (size 1.27 1.27)))
     )
@@
       (project "MuscleRecoveryV1"
         (path "/4e550305-79d2-4e4a-a502-817ebcc79f9a/50c43c35-6798-4b23-b9a6-29e92679e65f"
-          (reference "IC2") (unit 1)
+          (reference "U10") (unit 1)
         )
       )
