File: production/ecad/MuscleRecoveryV2 Copy/MuscleEMG.kicad_sch (KiCad schematic)
At the start: 41 parts, among them J1 AudioJack3, J2 Screw_Terminal_01x03, J5 Screw_Terminal_01x10, U5 AD8232ACPZ-R7, U7 ADS1115IDGS

Commit message: Created New Layout
Parts:
- removed J2: Screw_Terminal_01x03, symbol Connector:Screw_Terminal_01x03
- removed J5: Screw_Terminal_01x10, symbol Connector:Screw_Terminal_01x10
- C1, C10, C11, C14, C2, C3, C4: footprint Capacitor_SMD:C_0805_2012Metric -> Capacitor_SMD:C_0402_1005Metric
- D5, D6: footprint LED_THT:LED_D1.8mm_W3.3mm_H2.4mm -> LED_SMD:LED_0402_1005Metric
- J1: footprint (none) -> Muscle_Recovery_Footprint_Library:CUI_SJ-3523-SMT-TR
- R1, R19, R2, R20, R21, R22, R23, R24, R25, R26, R28, R29, R3, R4, R5, R6, R61, R62, R63, R64, R7: footprint Resistor_SMD:R_0805_2012Metric -> Resistor_SMD:R_0402_1005Metric
- R44, R45, R46, R47, R48, R49: footprint Resistor_SMD:R_0805_2012Metric -> Resistor_SMD:R_01005_0402Metric
- U5: footprint AD8232ACPZ-R7:CP_20_10_ADI -> Muscle_Recovery_Footprint_Library:LFCSP_20

Commit message: Pushing Layout Changes for Andy's Layout
Parts:
- R44, R45, R46, R47, R48, R49: footprint Resistor_SMD:R_01005_0402Metric -> Resistor_SMD:R_0402_1005Metric
Changed lines of the file:
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@@
       (effects (font (size 1.27 1.27)))
     )
-    (property "Footprint" "Resistor_SMD:R_01005_0402Metric" (at 66.04 171.958 90)
+    (property "Footprint" "Resistor_SMD:R_0402_1005Metric" (at 66.04 171.958 90)
       (effects (font (size 1.27 1.27)) hide)
     )
@@
       (effects (font (size 1.27 1.27)))
     )
-    (property "Footprint" "Resistor_SMD:R_01005_0402Metric" (at 138.43 24.638 90)
+    (property "Footprint" "Resistor_SMD:R_0402_1005Metric" (at 138.43 24.638 90)
       (effects (font (size 1.27 1.27)) hide)
     )
@@
       (effects (font (size 1.27 1.27)))
     )
-    (property "Footprint" "Resistor_SMD:R_01005_0402Metric" (at 121.92 24.638 90)
+    (property "Footprint" "Resistor_SMD:R_0402_1005Metric" (at 121.92 24.638 90)
       (effects (font (size 1.27 1.27)) hide)
     )
@@
       (effects (font (size 1.27 1.27)))
     )
-    (property "Footprint" "Resistor_SMD:R_01005_0402Metric" (at 66.04 174.498 90)
+    (property "Footprint" "Resistor_SMD:R_0402_1005Metric" (at 66.04 174.498 90)
       (effects (font (size 1.27 1.27)) hide)
     )
@@
       (effects (font (size 1.27 1.27)))
     )
-    (property "Footprint" "Resistor_SMD:R_01005_0402Metric" (at 144.78 107.188 90)
+    (property "Footprint" "Resistor_SMD:R_0402_1005Metric" (at 144.78 107.188 90)
       (effects (font (size 1.27 1.27)) hide)
     )
@@
       (effects (font (size 1.27 1.27)))
     )
-    (property "Footprint" "Resistor_SMD:R_01005_0402Metric" (at 62.23 166.878 90)
-      (effects (font (size 1.27 1.27)) hide)
-    )
+    (property "Footprint" "Resistor_SMD:R_0402_1005Metric" (at 62.23 166.878 90)
+      (effects (font (size 1.27 1.27)) hide)
+    )

Commit message: Committing My pliminary placement for my PCB <3
Parts:
- removed J1: AudioJack3, Muscle_Recovery_Footprint_Library:CUI_SJ-3523-SMT-TR, symbol Connector_Audio:AudioJack3
- added J5: SJ1-3533NG, Muscle_Recovery_Footprint_Library:CUI_SJ1-3533NG, symbol MuscleRecoverySymbolLibray:SJ1-3533NG
Connections:
- net LA: now also J5.1
- net RA: now also J5.3
- net RL: now also J5.2
Changed lines of the file:
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@@
     (effects (font (size 1.27 1.27)) (justify left bottom))
   )
-  (text "Audiojack. Connections must be configured." (at 16.51 53.34 0)
+  (text "Audiojack. Connections must be configured." (at 19.685 36.83 0)
     (effects (font (size 1.27 1.27)) (justify left bottom))
   )
@@
     (effects (font (size 5 5) bold) (justify left bottom))
   )
-  (global_label "RA" (shape input) (at 35.56 63.5 0) (fields_autoplaced)
-    (effects (font (size 1.27 1.27)) (justify left))
-    (property "Intersheetrefs" "${INTERSHEET_REFS}" (at 40.9038 63.5 0)
+  (global_label "RA" (shape input) (at 52.07 50.165 0) (fields_autoplaced)
+    (effects (font (size 1.27 1.27)) (justify left))
+    (property "Intersheetrefs" "${INTERSHEET_REFS}" (at 57.4138 50.165 0)
       (effects (font (size 1.27 1.27)) (justify left) hide)
     )
@@
     )
   )
-  (global_label "RL" (shape input) (at 35.56 66.04 0) (fields_autoplaced)
-    (effects (font (size 1.27 1.27)) (justify left))
-    (property "Intersheetrefs" "${INTERSHEET_REFS}" (at 40.8433 66.04 0)
+  (global_label "RL" (shape input) (at 52.07 52.705 0) (fields_autoplaced)
+    (effects (font (size 1.27 1.27)) (justify left))
+    (property "Intersheetrefs" "${INTERSHEET_REFS}" (at 57.3533 52.705 0)
       (effects (font (size 1.27 1.27)) (justify left) hide)
     )
@@
     )
   )
-  (global_label "LA" (shape input) (at 35.56 60.96 0) (fields_autoplaced)
-    (effects (font (size 1.27 1.27)) (justify left))
-    (property "Intersheetrefs" "${INTERSHEET_REFS}" (at 40.6619 60.96 0)
+  (global_label "LA" (shape input) (at 52.07 47.625 0) (fields_autoplaced)
+    (effects (font (size 1.27 1.27)) (justify left))
+    (property "Intersheetrefs" "${INTERSHEET_REFS}" (at 57.1719 47.625 0)
       (effects (font (size 1.27 1.27)) (justify left) hide)
     )
@@
     )
   )
+  (symbol (lib_id "MuscleRecoverySymbolLibray:SJ1-3533NG") (at 36.83 50.165 0) (unit 1)
+    (in_bom yes) (on_board yes) (dnp no) (fields_autoplaced)
+    (property "Reference" "J5" (at 36.83 40.005 0)
+      (effects (font (size 1.27 1.27)))
+    )
+    (property "Value" "SJ1-3533NG" (at 36.83 42.545 0)
+      (effects (font (size 1.27 1.27)))
+    )
+    (property "Footprint" "Muscle_Recovery_Footprint_Library:CUI_SJ1-3533NG" (at 36.83 50.165 0)
+      (effects (font (size 1.27 1.27)) (justify left bottom) hide)
+    )
+    (property "Datasheet" "" (at 36.83 50.165 0)
+      (effects (font (size 1.27 1.27)) (justify left bottom) hide)
+    )
+    (property "MF" "CUI Devices" (at 36.83 50.165 0)
+      (effects (font (size 1.27 1.27)) (justify left bottom) hide)
+    )
+    (property "DESCRIPTION" "3.5 mm, Stereo, Right Angle, Through Hole, Isolated Ground, Audio Jack Connector" (at 36.83 50.165 0)
+      (effects (font (size 1.27 1.27)) (justify left bottom) hide)
+    )
+    (property "PACKAGE" "None" (at 36.83 50.165 0)
+      (effects (font (size 1.27 1.27)) (justify left bottom) hide)
+    )
+    (property "PRICE" "None" (at 36.83 50.165 0)
+      (effects (font (size 1.27 1.27)) (justify left bottom) hide)
+    )
+    (property "CUI_PURCHASE_URL" "https://www.cuidevices.com/product/interconnect/connectors/audio-connectors/jacks/sj1-353xng-series?utm_source=snapeda.com&utm_medium=referral&utm_campaign=snapedaBOM" (at 36.83 50.165 0)
+      (effects (font (size 1.27 1.27)) (justify left bottom) hide)
+    )
+    (property "MP" "SJ1-3533NG" (at 36.83 50.165 0)
+      (effects (font (size 1.27 1.27)) (justify left bottom) hide)
+    )
+    (property "AVAILABILITY" "Unavailable" (at 36.83 50.165 0)
+      (effects (font (size 1.27 1.27)) (justify left bottom) hide)
+    )
+    (pin "1")
+    (pin "2")
+    (pin "3")
+    (instances
+      (project "MuscleRecoveryV1"
+        (path "/4e550305-79d2-4e4a-a502-817ebcc79f9a/284c60dd-e199-4b03-b99f-cc7eaed256f8"
+          (reference "J5") (unit 1)
+        )
+      )
+    )
+  )
   (symbol (lib_id "Analog_ADC:ADS1115IDGS") (at 45.72 170.18 0) (unit 1)
     (in_bom yes) (on_board yes) (dnp no) (fields_autoplaced)
@@
         )
       )
-    )
-  )
-  (symbol (lib_id "Connector_Audio:AudioJack3") (at 30.48 63.5 0) (unit 1)
-    (in_bom yes) (on_board yes) (dnp no) (fields_autoplaced)
-    (property "Reference" "J1" (at 28.575 54.61 0)
-      (effects (font (size 1.27 1.27)))
-    )
-    (property "Value" "AudioJack3" (at 28.575 57.15 0)
-      (effects (font (size 1.27 1.27)))
-    )
-    (property "Footprint" "Muscle_Recovery_Footprint_Library:CUI_SJ-3523-SMT-TR" (at 30.48 63.5 0)
-      (effects (font (size 1.27 1.27)) hide)
-    )
-    (property "Datasheet" "~" (at 30.48 63.5 0)
-      (effects (font (size 1.27 1.27)) hide)
-    )
-    (pin "R")
-    (pin "S")
-    (pin "T")
-    (instances
-      (project "MuscleRecoveryV1"
-        (path "/4e550305-79d2-4e4a-a502-817ebcc79f9a/284c60dd-e199-4b03-b99f-cc7eaed256f8"
-          (reference "J1") (unit 1)
-        )
-      )

Commit message: committing some recent changes to layout
Parts:
- removed J5: SJ1-3533NG, Muscle_Recovery_Footprint_Library:CUI_SJ1-3533NG, symbol MuscleRecoverySymbolLibray:SJ1-3533NG
- removed R29: 4.7k, Resistor_SMD:R_0402_1005Metric, symbol Device:R
- removed R47, R48, R49: 0, Resistor_SMD:R_0402_1005Metric, symbol Device:R
- removed R61: DNP, Resistor_SMD:R_0402_1005Metric, symbol Device:R
- added J6: Screw_Terminal_01x03, Connector_PinHeader_2.54mm:PinHeader_1x03_P2.54mm_Horizontal, symbol Connector:Screw_Terminal_01x03
Connections:
- net ALERT/READY: now also U7.2 (ALERT/RDY)
- net LA: now also J6.3 (Pin_3)
- net RA: now also J6.2 (Pin_2)
- net RL: now also J6.1 (Pin_1)
- net SCL: now also U7.10 (SCL)
- net SDA: now also U7.9 (SDA)

Commit message: Pushing Most of the final changes for PCB REV2
Parts:
- removed J6: Screw_Terminal_01x03, Connector_PinHeader_2.54mm:PinHeader_1x03_P2.54mm_Horizontal, symbol Connector:Screw_Terminal_01x03
- added J2: SM03B-SRSS-TB_LF__SN_, Muscle_Recovery_Footprint_Library:JST_SM03B-SRSS-TB_LF__SN_, symbol MuscleRecoverySymbolLibray:SM03B-SRSS-TB_LF__SN_
Connections:
- net LA: now also J2.2
- net RA: now also J2.3
- net RL: now also J2.1
- new net: J2.S1 (SHIELD), J2.S2 (SHIELD)
- no-connect marks 3 -> 4
Changed lines of the file:
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@@
   (no_connect (at 35.56 172.72))
   (no_connect (at 35.56 170.18))
+  (no_connect (at 52.07 60.96))
   (wire (pts (xy 119.38 52.07) (xy 119.38 49.53))
     (stroke (width 0) (type default))
@@
     (stroke (width 0) (type default))
   )
+  (wire (pts (xy 52.07 55.88) (xy 60.96 55.88))
+    (stroke (width 0) (type default))
+  )
   (wire (pts (xy 219.71 52.07) (xy 245.11 52.07))
     (stroke (width 0) (type default))
@@
     (stroke (width 0) (type default))
   )
+  (wire (pts (xy 52.07 53.34) (xy 60.96 53.34))
+    (stroke (width 0) (type default))
+  )
   (wire (pts (xy 119.38 35.56) (xy 124.46 35.56))
     (stroke (width 0) (type default))
@@
   )
   (wire (pts (xy 125.73 22.86) (xy 128.27 22.86))
+    (stroke (width 0) (type default))
+  )
+  (wire (pts (xy 52.07 50.8) (xy 60.96 50.8))
     (stroke (width 0) (type default))
   )
@@
   (text "ADC" (at 25.4 139.7 0)
     (effects (font (size 5 5) bold) (justify left bottom))
-  )
-  (global_label "RA" (shape input) (at 52.07 50.165 0) (fields_autoplaced)
-    (effects (font (size 1.27 1.27)) (justify left))
-    (property "Intersheetrefs" "${INTERSHEET_REFS}" (at 57.4138 50.165 0)
-      (effects (font (size 1.27 1.27)) (justify left) hide)
-    )
   )
   (global_label "SCL" (shape input) (at 76.2 170.18 0) (fields_autoplaced)
@@
     )
   )
+  (global_label "LA" (shape input) (at 60.96 53.34 0) (fields_autoplaced)
+    (effects (font (size 1.27 1.27)) (justify left))
+    (property "Intersheetrefs" "${INTERSHEET_REFS}" (at 66.0619 53.34 0)
+      (effects (font (size 1.27 1.27)) (justify left) hide)
+    )
+  )
   (global_label "SW" (shape input) (at 144.78 66.04 180) (fields_autoplaced)
     (effects (font (size 1.27 1.27)) (justify right))
@@
     )
   )
-  (global_label "RL" (shape input) (at 52.07 52.705 0) (fields_autoplaced)
-    (effects (font (size 1.27 1.27)) (justify left))
-    (property "Intersheetrefs" "${INTERSHEET_REFS}" (at 57.3533 52.705 0)
-      (effects (font (size 1.27 1.27)) (justify left) hide)
-    )
-  )
   (global_label "ALERT{slash}READY" (shape bidirectional) (at 226.06 156.21 180) (fields_autoplaced)
     (effects (font (size 1.27 1.27)) (justify right))
@@
     )
   )
-  (global_label "LA" (shape input) (at 52.07 47.625 0) (fields_autoplaced)
+  (global_label "RA" (shape input) (at 60.96 55.88 0) (fields_autoplaced)
     (effects (font (size 1.27 1.27)) (justify left))
-    (property "Intersheetrefs" "${INTERSHEET_REFS}" (at 57.1719 47.625 0)
+    (property "Intersheetrefs" "${INTERSHEET_REFS}" (at 66.3038 55.88 0)
       (effects (font (size 1.27 1.27)) (justify left) hide)
     )
@@
     )
   )
+  (global_label "RL" (shape input) (at 60.96 50.8 0) (fields_autoplaced)
+    (effects (font (size 1.27 1.27)) (justify left))
+    (property "Intersheetrefs" "${INTERSHEET_REFS}" (at 66.2433 50.8 0)
+      (effects (font (size 1.27 1.27)) (justify left) hide)
+    )
+  )
   (global_label "LOD+" (shape input) (at 219.71 71.12 0) (fields_autoplaced)
     (effects (font (size 1.27 1.27)) (justify left))
@@
         (path "/4e550305-79d2-4e4a-a502-817ebcc79f9a/284c60dd-e199-4b03-b99f-cc7eaed256f8"
           (reference "C3") (unit 1)
-        )
-      )
-    )
-  )
-  (symbol (lib_id "Connector:Screw_Terminal_01x03") (at 46.99 50.165 180) (unit 1)
-    (in_bom yes) (on_board yes) (dnp no) (fields_autoplaced)
-    (property "Reference" "J6" (at 46.99 41.91 0)
-      (effects (font (size 1.27 1.27)))
-    )
-    (property "Value" "Screw_Terminal_01x03" (at 46.99 44.45 0)
-      (effects (font (size 1.27 1.27)))
-    )
-    (property "Footprint" "Connector_PinHeader_2.54mm:PinHeader_1x03_P2.54mm_Horizontal" (at 46.99 50.165 0)
-      (effects (font (size 1.27 1.27)) hide)
-    )
-    (property "Datasheet" "~" (at 46.99 50.165 0)
-      (effects (font (size 1.27 1.27)) hide)
-    )
-    (pin "1")
-    (pin "2")
-    (pin "3")
-    (instances
-      (project "MuscleRecoveryV1"
-        (path "/4e550305-79d2-4e4a-a502-817ebcc79f9a/284c60dd-e199-4b03-b99f-cc7eaed256f8"
-          (reference "J6") (unit 1)
         )
       )
@@
         )
       )
+    )
+  )
+  (symbol (lib_id "MuscleRecoverySymbolLibray:SM03B-SRSS-TB_LF__SN_") (at 41.91 55.88 0) (mirror y) (unit 1)
+    (in_bom yes) (on_board yes) (dnp no)
+    (property "Reference" "J2" (at 38.1 46.99 0)
+      (effects (font (size 1.27 1.27)) (justify left))
+    )
+    (property "Value" "SM03B-SRSS-TB_LF__SN_" (at 61.595 66.04 0)
+      (effects (font (size 1.27 1.27)) (justify left))
+    )
+    (property "Footprint" "Muscle_Recovery_Footprint_Library:JST_SM03B-SRSS-TB_LF__SN_" (at 34.29 71.12 0)
+      (effects (font (size 1.27 1.27)) (justify bottom) hide)
+    )
+    (property "Datasheet" "" (at 41.91 55.88 0)
+      (effects (font (size 1.27 1.27)) hide)
+    )
+    (property "MF" "JST Sales America Inc." (at 34.29 71.12 0)
+      (effects (font (size 1.27 1.27)) (justify bottom) hide)
+    )
+    (property "Description" "\nConnector Header Surface Mount, Right Angle 3 position 0.039 (1.00mm)\n" (at 34.29 71.12 0)
+      (effects (font (size 1.27 1.27)) (justify bottom) hide)
+    )
+    (property "Package" "None" (at 29.21 62.23 0)
+      (effects (font (size 1.27 1.27)) (justify bottom) hide)
+    )
+    (property "Price" "None" (at 26.67 62.23 0)
+      (effects (font (size 1.27 1.27)) (justify bottom) hide)
+    )
+    (property "Check_prices" "https://www.snapeda.com/parts/SM03B-SRSS-TB(LF)(SN)/JST+Sales+America+Inc./view-part/?ref=eda" (at 34.29 71.12 0)
+      (effects (font (size 1.27 1.27)) (justify bottom) hide)
+    )
+    (property "STANDARD" "Manufacturer Recommendation" (at 34.29 71.12 0)
+      (effects (font (size 1.27 1.27)) (justify bottom) hide)
+    )
+    (property "SnapEDA_Link" "https://www.snapeda.com/parts/SM03B-SRSS-TB(LF)(SN)/JST+Sales+America+Inc./view-part/?ref=snap" (at 34.29 71.12 0)
+      (effects (font (size 1.27 1.27)) (justify bottom) hide)
+    )
+    (property "MP" "SM03B-SRSS-TB(LF)(SN)" (at 34.29 71.12 0)
+      (effects (font (size 1.27 1.27)) (justify bottom) hide)
+    )
+    (property "Availability" "In Stock" (at 29.21 58.42 0)
+      (effects (font (size 1.27 1.27)) (justify bottom) hide)
+    )
+    (property "MANUFACTURER" "JST" (at 27.94 60.96 0)
+      (effects (font (size 1.27 1.27)) (justify bottom) hide)
+    )
+    (pin "1")
+    (pin "2")
+    (pin "3")
+    (pin "S1")
+    (pin "S2")
+    (instances
+      (project "MuscleRecoveryV1"
+        (path "/4e550305-79d2-4e4a-a502-817ebcc79f9a/284c60dd-e199-4b03-b99f-cc7eaed256f8"
+          (reference "J2") (unit 1)
+        )
+      )

Commit message: Pushing changes post schematic review
Parts:
- removed D5, D6: LED, LED_SMD:LED_0402_1005Metric, symbol Device:LED
- removed R24, R45, R63, R64: 0, Resistor_SMD:R_0402_1005Metric, symbol Device:R
- removed R28: 180, Resistor_SMD:R_0402_1005Metric, symbol Device:R
- removed R44: DNP, Resistor_SMD:R_0402_1005Metric, symbol Device:R
- removed R46: 1k, Resistor_SMD:R_0402_1005Metric, symbol Device:R
- added R24: 1K, symbol Device:R_Small
Connections:
- net +3V3: now also R20.2, R21.2, U5.15 (FR), R24.1
- net ALERT/READY: no longer U7.2 (ALERT/RDY)
- net GND: now also U5.14 (AC/*DC)
- net SDN: now also R24.2
- no-connect marks 4 -> 5
Other:
- note added: "0x48"

Commit message: Pushing final Rev2 PCBA Files
Parts:
- R24: footprint (none) -> Resistor_SMD:R_0402_1005Metric
Connections:
- net at J2.S1 (SHIELD): no longer J2.S2 (SHIELD)
- no-connect marks 5 -> 6
Changed lines of the file:
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@@
   (no_connect (at 55.88 165.1))
   (no_connect (at 35.56 170.18))
+  (no_connect (at 52.07 58.42))
   (no_connect (at 52.07 60.96))
   (wire (pts (xy 119.38 52.07) (xy 119.38 49.53))
@@
       (effects (font (size 1.27 1.27)) (justify left))
     )
-    (property "Footprint" "" (at 232.41 74.93 0)
-      (effects (font (size 1.27 1.27)) hide)
-    )
+    (property "Footprint" "Resistor_SMD:R_0402_1005Metric" (at 232.41 74.93 0)
+      (effects (font (size 1.27 1.27)) hide)
+    )
