File: production/ecad/MuscleRecoveryV2 Copy/MuscleRecoveryV1.kicad_pcb (KiCad board)
At the start: 4 copper layers, 42 x 39 mm, 110 parts, among them IC2 W25Q128JVPIQ, J1 S2B-PH-SM4-TB_LF__SN_, J2 SM03B-SRSS-TB_LF__SN_, J3 SM02B-SRSS-TB_LF__SN_, J4 SM02B-SRSS-TB_LF__SN_, J5 USB4110-GF-A, J7 51296-1894, J8 SM02B-SRSS-TB_LF__SN_, Q1 FDN340P, Q2 AO3400A, Q3 AO3400A, Q4 AO3400A, U1 AP1117-33, U2 MCP73831-2-OT, U3 CP2102N-Axx-xQFN28, U4 PCF8523T/1_118, U5 AD8232ACPZ-R7, U6 ESP32-WROOM-32E__16MB_, U7 ADS1115IDGS, U8 ADXL343, U9 MAX17043G+T, Y1 ABS07-32.768KHZ-7-T

Commit message: Final Final FInal PCB
Parts:
- renumbered IC2 to U10
Changed lines of the file:
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@@
     (property "ki_description" "128M-bit Serial Flash Memory with uniform 4KB sectors and Dual/Quad SPI")
     (attr smd)
-    (fp_text reference "IC2" (at 2.794 -3.429 180) (layer "B.SilkS")
+    (fp_text reference "U10" (at 2.794 -3.429 180) (layer "B.SilkS")
         (effects (font (size 0.762 0.762) (thickness 0.1905)) (justify mirror))
     )
@@
   (segment (start 189.302 78.613) (end 190.119 77.796) (width 0.127) (layer "F.Cu") (net 1))
   (segment (start 191.065 66.032) (end 191.84 66.032) (width 0.1905) (layer "F.Cu") (net 1))
+  (segment (start 190.119 76.708) (end 190.881 75.946) (width 0.1905) (layer "F.Cu") (net 1))
   (segment (start 187.833 78.613) (end 189.302 78.613) (width 0.127) (layer "F.Cu") (net 1))
   (segment (start 166.356 57.369) (end 167.986 57.369) (width 0.1905) (layer "F.Cu") (net 1))
-  (segment (start 190.119 76.708) (end 189.992 76.581) (width 0.1905) (layer "F.Cu") (net 1))
+  (segment (start 190.881 75.754) (end 190.43 75.303) (width 0.1905) (layer "F.Cu") (net 1))
   (segment (start 166.356 57.369) (end 164.053 57.369) (width 0.1905) (layer "F.Cu") (net 1))
   (segment (start 187.957 63.249) (end 188.849 62.357) (width 0.1905) (layer "F.Cu") (net 1))
@@
   (segment (start 187.957 63.754) (end 187.957 63.249) (width 0.1905) (layer "F.Cu") (net 1))
   (segment (start 167.986 57.369) (end 168.021 57.404) (width 0.1905) (layer "F.Cu") (net 1))
-  (segment (start 189.992 76.581) (end 189.992 75.741) (width 0.1905) (layer "F.Cu") (net 1))
+  (segment (start 190.119 77.796) (end 190.119 76.708) (width 0.1905) (layer "F.Cu") (net 1))
   (segment (start 159.709 65.221) (end 159.709 65.667) (width 0.1905) (layer "F.Cu") (net 1))
-  (segment (start 189.992 75.741) (end 190.43 75.303) (width 0.1905) (layer "F.Cu") (net 1))
   (segment (start 187.325 62.484) (end 186.946 62.484) (width 0.1905) (layer "F.Cu") (net 1))
-  (segment (start 190.119 77.796) (end 190.119 76.708) (width 0.1905) (layer "F.Cu") (net 1))
+  (segment (start 190.881 75.946) (end 190.881 75.754) (width 0.1905) (layer "F.Cu") (net 1))
   (segment (start 187.96 58.674) (end 186.946 58.674) (width 0.1905) (layer "F.Cu") (net 1))
   (segment (start 192.405 64.262) (end 191.897 63.754) (width 0.1905) (layer "F.Cu") (net 1))
@@
   (segment (start 193.36 74.706) (end 194.31 73.756) (width 0.127) (layer "B.Cu") (net 39))
   (segment (start 194.31 73.756) (end 194.31 72.263) (width 0.127) (layer "B.Cu") (net 39))
-  (segment (start 184.912 86.36) (end 191.897 86.36) (width 0.127) (layer "B.Cu") (net 40))
+  (segment (start 184.912 86.36) (end 191.978448 86.36) (width 0.127) (layer "B.Cu") (net 40))
   (segment (start 195.78 82.558448) (end 195.78 75.226) (width 0.127) (layer "B.Cu") (net 40))
   (segment (start 184.772 86.22) (end 184.912 86.36) (width 0.127) (layer "B.Cu") (net 40))
   (segment (start 195.78 75.226) (end 195.26 74.706) (width 0.127) (layer "B.Cu") (net 40))
-  (segment (start 192.486448 85.852) (end 195.78 82.558448) (width 0.127) (layer "B.Cu") (net 40))
-  (segment (start 192.405 85.852) (end 192.486448 85.852) (width 0.127) (layer "B.Cu") (net 40))
-  (segment (start 191.897 86.36) (end 192.405 85.852) (width 0.127) (layer "B.Cu") (net 40))
+  (segment (start 191.978448 86.36) (end 195.78 82.558448) (width 0.127) (layer "B.Cu") (net 40))
   (segment (start 184.772 84.595) (end 184.772 86.22) (width 0.127) (layer "B.Cu") (net 40))
   (segment (start 188.47 70.231) (end 188.47 69.598) (width 0.1905) (layer "F.Cu") (net 41))
@@
   (segment (start 184.8612 78.232) (end 184.8612 78.8162) (width 0.127) (layer "B.Cu") (net 47))
   (segment (start 185.272 79.227) (end 185.272 79.695) (width 0.127) (layer "B.Cu") (net 47))
+  (segment (start 191.897 79.121) (end 192.659 79.883) (width 0.127) (layer "F.Cu") (net 48))
   (segment (start 191.951 86.433) (end 186.509 86.433) (width 0.127) (layer "F.Cu") (net 48))
-  (segment (start 186.946 61.214) (end 192.913 61.214) (width 0.127) (layer "F.Cu") (net 48))
-  (segment (start 192.913 61.214) (end 193.167 61.468) (width 0.127) (layer "F.Cu") (net 48))
-  (segment (start 193.167 71.501) (end 193.167 76.41909) (width 0.127) (layer "F.Cu") (net 48))
+  (segment (start 193.421 71.647) (end 193.421 76.16509) (width 0.127) (layer "F.Cu") (net 48))
+  (segment (start 193.421 67.618) (end 193.221 67.818) (width 0.127) (layer "F.Cu") (net 48))
   (segment (start 194.637 81.334) (end 194.637 83.747) (width 0.127) (layer "F.Cu") (net 48))
   (segment (start 194.818 80.01) (end 194.818 81.153) (width 0.127) (layer "F.Cu") (net 48))
   (segment (start 194.637 83.747) (end 191.951 86.433) (width 0.127) (layer "F.Cu") (net 48))
   (segment (start 185.547 85.979) (end 185.547 85.598) (width 0.127) (layer "F.Cu") (net 48))
-  (segment (start 191.897 79.121) (end 192.659 79.883) (width 0.127) (layer "F.Cu") (net 48))
+  (segment (start 193.221 71.447) (end 193.421 71.647) (width 0.127) (layer "F.Cu") (net 48))
+  (segment (start 193.167 65.659) (end 193.421 65.913) (width 0.127) (layer "F.Cu") (net 48))
+  (segment (start 192.913 61.214) (end 193.167 61.468) (width 0.127) (layer "F.Cu") (net 48))
   (segment (start 185.674 86.106) (end 185.547 85.979) (width 0.127) (layer "F.Cu") (net 48))
-  (segment (start 193.221 71.447) (end 193.167 71.501) (width 0.127) (layer "F.Cu") (net 48))
-  (segment (start 193.167 76.41909) (end 191.897 77.68909) (width 0.127) (layer "F.Cu") (net 48))
   (segment (start 193.421 65.913) (end 193.421 67.618) (width 0.127) (layer "F.Cu") (net 48))
-  (segment (start 191.897 77.68909) (end 191.897 79.121) (width 0.127) (layer "F.Cu") (net 48))
   (segment (start 186.509 86.433) (end 186.182 86.106) (width 0.127) (layer "F.Cu") (net 48))
   (segment (start 186.182 86.106) (end 185.674 86.106) (width 0.127) (layer "F.Cu") (net 48))
-  (segment (start 193.221 67.818) (end 193.221 71.447) (width 0.127) (layer "F.Cu") (net 48))
-  (segment (start 193.167 61.468) (end 193.167 65.659) (width 0.127) (layer "F.Cu") (net 48))
   (segment (start 194.818 81.153) (end 194.637 81.334) (width 0.127) (layer "F.Cu") (net 48))
-  (segment (start 193.421 67.618) (end 193.221 67.818) (width 0.127) (layer "F.Cu") (net 48))
-  (segment (start 193.167 65.659) (end 193.421 65.913) (width 0.127) (layer "F.Cu") (net 48))
+  (segment (start 191.897 77.68909) (end 191.897 79.121) (width 0.127) (layer "F.Cu") (net 48))
+  (segment (start 193.421 76.16509) (end 191.897 77.68909) (width 0.127) (layer "F.Cu") (net 48))
+  (segment (start 186.946 61.214) (end 192.913 61.214) (width 0.127) (layer "F.Cu") (net 48))
+  (segment (start 193.167 61.468) (end 193.167 65.659) (width 0.127) (layer "F.Cu") (net 48))
+  (segment (start 193.221 67.818) (end 193.221 71.447) (width 0.127) (layer "F.Cu") (net 48))
   (via (at 192.659 79.883) (size 0.6) (drill 0.3) (layers "F.Cu" "B.Cu") (net 48))
   (via (at 194.818 80.01) (size 0.6) (drill 0.3) (layers "F.Cu" "B.Cu") (net 48))
